File: Electrical/Main Board/DebuggingBoard.kicad_sch (KiCad schematic)
At the start: 81 parts, among them J1 Conn_01x05_Socket, J2 Conn_01x08_Socket, J3 Conn_01x01_Socket, SW1 SW_SPDT, U1 STM32F373CCTx, U2 AP62300TWU, U3 ADS7056IRUGR, U4 ADG1414BRU, U6 LM27761, U7 OPA2156xD, U8 TPS7A9401DSCR, Y1 16MHz

Commit message: updated main:
Parts:
- removed C12: 10pF, symbol Device:C
- removed C15, C18, C21, C25, C32, C34: 1uF, symbol Device:C
- removed C19, C20, C24, C31, C33: 100nF, symbol Device:C
- removed C22, C23: 10nF, symbol Device:C
- removed C28, C29: 4.7uF, symbol Device:C
- removed C30: 2.2uF, symbol Device:C
- removed C35: 680pF, symbol Device:C
- removed D1, D2: D, symbol Device:D
- removed F1: Fuse, symbol Device:Fuse
- removed J3: Conn_01x01_Socket, symbol Connector:Conn_01x01_Socket
- removed R10, R11, R13, R14: 20K, symbol Device:R
- removed R12, R7, R8, R9: 10K, symbol Device:R
- removed R15, R16, R17: 33R, symbol Device:R
- removed R20: 100K, symbol Device:R
- removed R21, R4: 10M, symbol Device:R
- removed R27, R5: 1M, symbol Device:R
- removed R6: 56.2K, symbol Device:R
- removed RV1: Varistor, symbol Device:Varistor
- removed U1: STM32F373CCTx, Package_QFP:LQFP-48_7x7mm_P0.5mm, symbol MCU_ST_STM32F3:STM32F373CCTx
- removed U3: ADS7056IRUGR, Rocketry_Easyeda:X2QFN-8_L1.5-W1.5-P0.50-BL, symbol ROCKETRY_EASYEDA:ADS7056IRUGR
- removed U4: ADG1414BRU, Package_SO:TSSOP-24_4.4x7.8mm_P0.65mm, symbol Analog_Switch:ADG1414BRU
- removed U6: LM27761, Package_SON:WSON-8-1EP_2x2mm_P0.5mm_EP0.9x1.6mm, symbol Regulator_SwitchedCapacitor:LM27761
- removed U7: OPA2156xD, Package_SO:SOIC-8_3.9x4.9mm_P1.27mm, symbol Amplifier_Operational:OPA2156xD
- added U1: STM32F446VETx, Package_QFP:LQFP-100_14x14mm_P0.5mm, symbol MCU_ST_STM32F4:STM32F446VETx
- C1: value 4.7uF -> 10uF
- C10, C5, C8: value 1uF -> 100nF
- C11: value 10pF -> 100nF
- C6, C7: value 10nF -> 100nF
- C9: value 10nF -> 10uF
- Y1: value 16MHz -> Crystal_GND24; footprint Crystal:Crystal_SMD_3225-4Pin_3.2x2.5mm -> (none)
Connections:
- net +3.3V: now also U1.100 (VDD), U1.11 (VDD), U1.19 (VDD), U1.28 (VDD), U1.50 (VDD), U1.6 (VBAT), U1.75 (VDD); no longer C10.1, C9.1
- net BOOT0: now also U1.94 (BOOT0)
- net GND: now also U1.10 (VSS), U1.20 (VSSA), U1.27 (VSS), U1.49 (VSS), U1.74 (VSS), U1.99 (VSS)
- net nRST: now also U1.14 (NRST)
- net OSC_OUT: now reaches Y1.3
- net OSC_OUT: now also U1.13 (PH1)
- net +3.3VA: now reaches C11.1
- net +3.3VA: now also C10.1, C9.1, U1.21 (VREF+), U1.22 (VDDA); no longer Y1.1
- new net OSC_IN: U1.12 (PH0), Y1.1
- no-connect marks 3 -> 2
Other:
- note added: "STM32F446"
- note removed: "0-3.6V"
- note removed: "0-360V"
- note removed: "0-36V"
- note removed: "ADC IC"
- note removed: "Inverting Supply -3.3V"
- note removed: "Multimeter Stuffs"
- note removed: "Op-Amp Mapping (+-20V -> 0 to 2.5V)"
- note removed: "Op-Amp Power Supply"
- note removed: "S1, S2, and S3 are used for ohmmeter S4, S5, and S6 are used for voltmeter S7, and S8 is used for ammeter"
- note removed: "STM32F373"
- moved on the sheet: C13, C14, C16, C17, C26, J1, J2, L1, R1, R18, R19, R2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

Commit message: VPSU and PMS complete
Parts:
- removed C13: 100n, Capacitor_SMD:C_0402_1005Metric, symbol Device:C
- removed C13: 10uF, Capacitor_SMD:C_0603_1608Metric, symbol Device:C
- removed C14 (x2): 22uF, Capacitor_SMD:C_0805_2012Metric, symbol Device:C
- removed C16, C17: 10uF, symbol Device:C
- removed C26: 4.7uF, symbol Device:C
- removed L1: FNR5020S3R3NT, Rocketry_Easyeda:IND-SMD_L5.0-W5.0_FNR50XXS, symbol Rocketry:FNR5020S3R3NT
- removed R1, R2: 5.1k, symbol Device:R
- removed R18: 10K, Resistor_SMD:R_0402_1005Metric, symbol Device:R
- removed R19: 37.4K, Resistor_SMD:R_0402_1005Metric, symbol Device:R
- removed R22: 316K, symbol Device:R
- removed R23: 100K, symbol Device:R
- removed R24: 12.4K, symbol Device:R
- removed R25: 187K, symbol Device:R
- removed U1: STM32F446VETx, Package_QFP:LQFP-100_14x14mm_P0.5mm, symbol MCU_ST_STM32F4:STM32F446VETx
- removed U2: AP62300TWU, Package_TO_SOT_SMD:TSOT-23-6, symbol Regulator_Switching:AP62300TWU
- removed U8: TPS7A9401DSCR, Rocketry_Easyeda:WSON-10_L3.0-W3.0-P0.50-TL-EP, symbol ROCKETRY_EASYEDA:TPS7A9401DSCR
- added C4, C7: 10pF, symbol Device:C
- added C44: 1uF, symbol Device:C
- added C45: 10uF, symbol Device:C
- added C46: 100nF, symbol Device:C
- added J1: Barrel_Jack_Switch, symbol Connector:Barrel_Jack_Switch
- added J4: Conn_01x02_Socket, symbol Connector:Conn_01x02_Socket
- added J5: Conn_01x03_Socket, symbol Connector:Conn_01x03_Socket
- added J6: Conn_01x04_Socket, symbol Connector:Conn_01x04_Socket
- added U1: STM32H563VGTx, Package_QFP:LQFP-100_14x14mm_P0.5mm, symbol MCU_ST_STM32H5:STM32H563VGTx
- added U6: CH224K, Package_SO:SSOP-10-1EP_3.9x4.9mm_P1mm_EP2.1x3.3mm, symbol Interface_USB:CH224K
- R26: value 22.1K -> 24K
- renumbered C7 to C10, C8 to C11, C10 to C12, C9 to C13, C11 to C2, C2 to C3, C3 to C5, C4 to C6, C5 to C8, C6 to C9, J1 to J2, J2 to J3
Connections:
- net LDO_VIN is gone; now on net +3.3V: J3.1 (Pin_1)
- net +3.3V: now also J5.1 (Pin_1), U1.100 (VDD), U1.11 (VDD), U1.22 (VDDA), U1.28 (VDD), U1.50 (VDD), U1.6 (VBAT), U1.75 (VDD)
- net +3.3VA: now also J5.2 (Pin_2), U1.21 (VREF+), U1.73 (VDDUSB)
- net BOOT0: now also U1.94 (BOOT0)
- net D+: now also U1.71 (PA12)
- net D-: now also U1.70 (PA11)
- net GND: now also R26.1, C44.2, C45.1, C46.1, J1.2, J1.3, J4.2 (Pin_2), J5.3 (Pin_3), U1.10 (VSS), U1.19 (VSSA), U1.20 (VREF-), U1.27 (VSS), U1.49 (VSS), U1.74 (VSS), U1.99 (VSS), U6.11 (GND); no longer R26.2
- net OSC_IN: now also C4.1, U1.12 (PH0)
- net OSC_OUT: now also C7.1, U1.13 (PH1)
- net SWCLK: now also U1.76 (PA14(JTCK)
- net SWDIO: now also U1.72 (PA13(JTMS)
- net nRST: now also U1.14 (NRST)
- net CC2: now reaches USB1.10 (CC2)
- net CC2: now also U6.6 (CC2)
- net CC1: now reaches USB1.4 (CC1)
- net CC1: now also U6.7 (CC1)
- net +5V renamed VBUS
- net VBUS: now also C45.2, C46.2, U6.8 (VBUS)
- new net: C44.1, U6.1 (VDD)
- new net: R26.2, U6.9 (CFG1)
- new net +12V: J1.1
- new net GND1: C4.2, C7.2
- new net USB_C_PG: U6.10 (PG)
- new net V_SELECT: J4.1 (Pin_1)
- no-connect marks 2 -> 8
Other:
- added sheet PowerManagement (PowerManagement.kicad_sch)
- note added: "12V Input"
- note added: "Oscilloscope Board Connectors"
- note added: "USB-C PD (12V)"
- note added: "Variable PSU Power Connector"
- note removed: "3.6V Switching Voltage Regulator"
- note removed: "Low-Noise 3.3V LDO"
- moved on the sheet: R3, SW1, USB1, Y1
