File: Electrical/Multimeter/MultimeterBoard/MultimeterBoard.kicad_sch (KiCad schematic)
At the start: 0 parts

Commit message: new layout
Parts:
- added U20: SM08B-PASS-TBT(LF)(SN), JLC_PARTS:CONN-SMD_SM08B-PASS-TBT-LF-SN, symbol JLC_PARTS:SM08B-PASS-TBT(LF)(SN)
Connections:
- new net ADC1_INP4: U20.1
- new net ADC2_INP8: U20.2
- new net BUZZER_CTRL: U20.8
- new net GND: U20.10, U20.3, U20.9
- new net R_SRC_100K: U20.5
- new net R_SRC_1K: U20.4
- new net V_RANGE_HIGH: U20.7
- new net V_RANGE_LOW: U20.6
Other:
- note added: "Multimeter Input"
