File: Electrical/MainBoard/DebuggingBoard.kicad_sch (KiCad schematic)
At the start: 30 parts, among them J1 Barrel_Jack_Switch, J2 Conn_01x05_Socket, J3 Conn_01x08_Socket, J4 Conn_01x02_Socket, J5 Conn_01x03_Socket, J6 Conn_01x04_Socket, SW1 SW_SPDT, U1 STM32H563VGTx, U6 CH224K, Y1 Crystal_GND24

Commit message: VPSU schem complete
Parts:
- added C53: 100nF, symbol Device:C
- added C54: 1nF, symbol Device:C
- added C55, C56: 2.2uF, symbol Device:C
- added C57, C58: 10uF, symbol Device:C
- added FB7, FB8: 600R@100MHz, symbol Device:FerriteBead
- C9: renamed from C45; value 10uF -> 4.7uF
- renumbered C9 to C10, C46 to C11, C44 to C12, C10 to C13, C11 to C14, C47 to C15, C12 to C16, C13 to C17, J4 to J3, J5 to J4, J6 to J5, J3 to J6, R26 to R1, R3 to R2, U6 to U1, U1 to U2
Connections:
- net +3.3V: now also U2.73 (VDDUSB), C58.1; no longer U2.22 (VDDA)
- net +3.3VA: now also C57.1, FB7.1, FB8.2; no longer C15.1, C16.1, C2.1, U2.21 (VREF+), U2.73 (VDDUSB)
- net GND: now also C53.2, C54.2, C55.2, C56.2, C57.2, C58.2
- net nRST: now also C53.1
- net at U2.48 (VCAP): now also C55.1
- net at U2.98 (VCAP): now also C56.1
- new net: C15.1, C16.1, FB7.2, U2.22 (VDDA)
- new net: C2.1, C54.1, FB8.1, U2.21 (VREF+)
Other:
- moved on the sheet: C1, C15, C16, C17, C2, J1, J2, J3, J4, J5, J6, R2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

Commit message: usb hs config
Parts:
- removed J5: Conn_01x04_Socket, symbol Connector:Conn_01x04_Socket
- removed U2: STM32H563VGTx, Package_QFP:LQFP-100_14x14mm_P0.5mm, symbol MCU_ST_STM32H5:STM32H563VGTx
- added C50: 10uF, symbol Device:C
- added C51, C52, C59, C60, C61: 100nF, symbol Device:C
- added C62, C63: 4.7uF, symbol Device:C
- added C64, C65: 15pF, symbol Device:C
- added J5: Conn_01x16_Socket, symbol Connector:Conn_01x16_Socket
- added NT2 (x2): NetTie_2, symbol Device:NetTie_2
- added R23: 12K, symbol Device:R
- added U2: STM32H723VGTx, Package_QFP:LQFP-100_14x14mm_P0.5mm, symbol MCU_ST_STM32H7:STM32H723VGTx
- added U3: USB3300-EZK, Package_DFN_QFN:QFN-32-1EP_5x5mm_P0.5mm_EP3.45x3.45mm, symbol Interface_USB:USB3300-EZK
- added Y2: X322524MOB4SI, symbol Device:Crystal_GND24
- Y1: value Crystal_GND24 -> X322525MOB4SI
Connections:
- net +3.3V: now also C50.1, C51.1, C52.1, C59.1, C60.1, C61.1, J5.15 (Pin_15), U2.100 (VDD), U2.11 (VDD), U2.27 (VDD), U2.50 (VDD), U2.6 (VBAT), U2.75 (VDD), U3.16 (VDD3.3), U3.25 (VDD3.3), U3.30 (VDD3.3), U3.31 (REG_EN), U3.6 (VDD3.3)
- net BOOT0: now also U2.94 (BOOT0)
- net D+: now also U3.7 (DP)
- net D-: now also U3.8 (DM)
- net GND: now also C50.2, C51.2, C52.2, C59.2, C60.2, C61.2, C62.2, C63.2, J5.1 (Pin_1), J5.16 (Pin_16), NT2.1, NT2.1, R23.2, U3.1 (GND), U3.2 (GND), U3.33 (GND)
- net GND1: now also C64.2, C65.2, NT2.2, NT2.2
- net OSC_IN: now also U2.12 (PH0)
- net OSC_OUT: now also U2.13 (PH1)
- net SWCLK: now also U2.76 (PA14(JTCK)
- net SWDIO: now also U2.72 (PA13(JTMS)
- net nRST: now also J5.14 (Pin_14), U2.14 (NRST)
- net at C15.1, C16.1, FB7.2: now also U2.21 (VDDA)
- net at C56.1: now also U2.73 (VCAP)
- net at C2.1, C54.1, FB8.1: now also U2.20 (VREF+)
- net at C55.1: now also U2.48 (VCAP)
- new net: C65.1, U3.28 (XI), Y2.1
- new net: C64.1, U3.27 (XO), Y2.3
- new net: C62.1, U3.15 (VDD1.8), U3.26 (VDD1.8)
- new net: R23.1, U3.32 (RBIAS)
- new net: C63.1, U3.29 (VDDA1.8)
- new net: U2.10 (VSS), U2.26 (VSS), U2.49 (VSS), U2.74 (VSS), U2.99 (VSS)
- new net FMC_A18: U2.60 (PD13)
- new net FMC_D0: U2.61 (PD14)
- new net FMC_D1: U2.62 (PD15)
- new net FMC_D10: U2.43 (PE13)
- new net FMC_D11: U2.44 (PE14)
- new net FMC_D12: U2.45 (PE15)
- new net FMC_D13: U2.55 (PD8)
- new net FMC_D14: U2.56 (PD9)
- new net FMC_D15: U2.57 (PD10)
- new net FMC_D2: U2.81 (PD0)
- new net FMC_D3: U2.82 (PD1)
- new net FMC_D4: U2.37 (PE7)
- new net FMC_D5: U2.38 (PE8)
- new net FMC_D6: U2.39 (PE9)
- new net FMC_D7: U2.40 (PE10)
- new net FMC_D8: U2.41 (PE11)
- new net FMC_D9: U2.42 (PE12)
- new net FMC_NE1: U2.88 (PD7)
- new net FMC_NOE: U2.85 (PD4)
- new net FMC_NWE: U2.86 (PD5)
- new net H723_RX: J5.13 (Pin_13)
- new net H723_TX: J5.12 (Pin_12)
- new net PSSI_D0: J5.2 (Pin_2), U2.63 (PC6)
- new net PSSI_D1: J5.3 (Pin_3), U2.64 (PC7)
- new net PSSI_D2: J5.4 (Pin_4), U2.65 (PC8)
- new net PSSI_D3: J5.5 (Pin_5), U2.66 (PC9)
- new net PSSI_D4: J5.6 (Pin_6), U2.3 (PE4)
- new net PSSI_D5: J5.7 (Pin_7), U2.84 (PD3)
- new net PSSI_D6: J5.8 (Pin_8), U2.4 (PE5)
- new net PSSI_D7: J5.9 (Pin_9), U2.5 (PE6)
- new net PSSI_DE: J5.11 (Pin_11), U2.28 (PA4)
- new net PSSI_PDCK: J5.10 (Pin_10), U2.30 (PA6)
- new net PSSI_RDY: U2.93 (PB7)
- new net ULPI_CK: U2.29 (PA5), U3.14 (CLKOUT)
- new net ULPI_D0: U2.25 (PA3), U3.24 (DATA0)
- new net ULPI_D1: U2.34 (PB0), U3.23 (DATA1)
- new net ULPI_D2: U2.35 (PB1), U3.22 (DATA2)
- new net ULPI_D3: U2.46 (PB10), U3.21 (DATA3)
- new net ULPI_D4: U2.47 (PB11), U3.20 (DATA4)
- new net ULPI_D5: U2.51 (PB12), U3.19 (DATA5)
- new net ULPI_D6: U2.52 (PB13), U3.18 (DATA6)
- new net ULPI_D7: U2.91 (PB5), U3.17 (DATA7)
- new net ULPI_DIR: U2.17 (PC2_C), U3.12 (DIR)
- new net ULPI_NXT: U2.18 (PC3_C), U3.11 (NXT)
- new net ULPI_RST: U3.9 (RESET)
- new net ULPI_STP: U2.15 (PC0), U3.13 (STP)
- new net USB_SOF: U2.67 (PA8)
- no-connect marks 8 -> 13
Other:
- note added: "GPIO Input"
- note added: "GPIO Output"
- note added: "USB High Speed External PHY"
- moved on the sheet: J1, J4, R2, SW1

Commit message: layout
Parts:
- removed C12: 1uF, symbol Device:C
- removed C3: 100nF, symbol Device:C
- removed C58: 10uF, symbol Device:C
- removed J5: Conn_01x16_Socket, symbol Connector:Conn_01x16_Socket
- removed NT2 (x2): NetTie_2, symbol Device:NetTie_2
- added C16: 1uF, Capacitor_SMD:C_0603_1608Metric, symbol Device:C
- added C22, C27: 10uF, Capacitor_SMD:C_0603_1608Metric, symbol Device:C
- added C25, C30, C36, C69: 100nF, Capacitor_SMD:C_0402_1005Metric, symbol Device:C
- added FB3: 100R@100MHz, Inductor_SMD:L_0805_2012Metric, symbol Device:FerriteBead
- added J5: Conn_02x12_Odd_Even, Connector_JST:JST_PUD_S24B-PUDSS-1_2x12_P2.00mm_Horizontal, symbol Connector_Generic:Conn_02x12_Odd_Even
- added R29: 10K, Resistor_SMD:R_0402_1005Metric, symbol Device:R
- added R3: 12K, Resistor_SMD:R_0402_1005Metric, symbol Device:R
- added R30: 1K, Resistor_SMD:R_0603_1608Metric, symbol Device:R
- added R5: 22R, Resistor_SMD:R_0402_1005Metric, symbol Device:R
- added U3: APS6404L-3SQR-ZR, Rocketry_Easyeda:USON-8_L3.0-W2.0-P0.50-BL-EP, symbol Rocketry_Easyeda:APS6404L-3SQR-ZR
- C1: renamed from C57; footprint (none) -> Capacitor_SMD:C_0603_1608Metric
- C10: renamed from C8; footprint (none) -> Capacitor_SMD:C_0402_1005Metric
- C11: renamed from C9; footprint (none) -> Capacitor_SMD:C_0603_1608Metric
- C12: renamed from C53; footprint (none) -> Capacitor_SMD:C_0402_1005Metric
- C13: renamed from C56; footprint (none) -> Capacitor_SMD:C_0603_1608Metric
- C14: renamed from C10; footprint (none) -> Capacitor_SMD:C_0402_1005Metric
- C15: renamed from C11; footprint (none) -> Capacitor_SMD:C_0402_1005Metric
- C17: renamed from C13; footprint (none) -> Capacitor_SMD:C_0402_1005Metric
- C18: renamed from C14; footprint (none) -> Capacitor_SMD:C_0402_1005Metric
- C19: renamed from C15; footprint (none) -> Capacitor_SMD:C_0402_1005Metric
- C2, C5: footprint (none) -> Capacitor_SMD:C_0402_1005Metric
- C20: renamed from C16; footprint (none) -> Capacitor_SMD:C_0402_1005Metric
- C21: renamed from C17; footprint (none) -> Capacitor_SMD:C_0603_1608Metric
- C23: renamed from C50; footprint (none) -> Capacitor_SMD:C_0603_1608Metric
- C24: renamed from C64; footprint (none) -> Capacitor_SMD:C_0402_1005Metric
- C26: renamed from C51; footprint (none) -> Capacitor_SMD:C_0402_1005Metric
- C28: renamed from C61; footprint (none) -> Capacitor_SMD:C_0402_1005Metric
- C29: renamed from C52; footprint (none) -> Capacitor_SMD:C_0402_1005Metric
- C3: renamed from C4; value 10pF -> 15pF; footprint (none) -> Capacitor_SMD:C_0402_1005Metric
- C31: renamed from C65; footprint (none) -> Capacitor_SMD:C_0402_1005Metric
- C32: renamed from C59; footprint (none) -> Capacitor_SMD:C_0402_1005Metric
- C33: renamed from C60; footprint (none) -> Capacitor_SMD:C_0402_1005Metric
- C34: renamed from C63; footprint (none) -> Capacitor_SMD:C_0603_1608Metric
- C35: renamed from C62; footprint (none) -> Capacitor_SMD:C_0603_1608Metric
- C4: renamed from C1; footprint (none) -> Capacitor_SMD:C_0603_1608Metric
- C6: renamed from C54; footprint (none) -> Capacitor_SMD:C_0402_1005Metric
- C7: renamed from C6; footprint (none) -> Capacitor_SMD:C_0402_1005Metric
- C8: renamed from C7; value 10pF -> 15pF; footprint (none) -> Capacitor_SMD:C_0402_1005Metric
- C9: renamed from C55; footprint (none) -> Capacitor_SMD:C_0603_1608Metric
- FB1: renamed from FB8; footprint (none) -> Inductor_SMD:L_0805_2012Metric
- FB2: renamed from FB7; footprint (none) -> Inductor_SMD:L_0805_2012Metric
- J1: footprint (none) -> Connector_BarrelJack:BarrelJack_Kycon_KLDX-0202-xC_Horizontal
- J2: footprint (none) -> Connector_JST:JST_PH_S5B-PH-K_1x05_P2.00mm_Horizontal
- J3: footprint (none) -> Connector_JST:JST_PH_S2B-PH-K_1x02_P2.00mm_Horizontal
- J4: renamed from J6; footprint (none) -> Connector_JST:JST_PH_S8B-PH-K_1x08_P2.00mm_Horizontal
- J6: renamed from J4; footprint (none) -> Connector_JST:JST_PH_S3B-PH-K_1x03_P2.00mm_Horizontal
- R1: footprint (none) -> Resistor_SMD:R_0603_1608Metric
- R2: footprint (none) -> Resistor_SMD:R_0402_1005Metric
- R4: renamed from R23; footprint (none) -> Resistor_SMD:R_0402_1005Metric
- SW1: footprint (none) -> Button_Switch_SMD:SW_SPDT_CK_JS102011SAQN
- Y1, Y2: footprint (none) -> Crystal:Crystal_SMD_3225-4Pin_3.2x2.5mm
- renumbered U3 to U4
Connections:
- net GND1 is gone; now on net GND: C24.2, C3.2, C31.2, C8.2
- net +3.3V: now also C22.1, C25.1, U3.8 (VDD)
- net +3.3VA: now also FB3.1; no longer J6.2 (Pin_2)
- net GND: now also U2.10 (VSS), U2.19 (VSSA), U2.26 (VSS), U2.49 (VSS), U2.74 (VSS), U2.99 (VSS), Y1.2, Y1.4, Y2.2, Y2.4, C16.1, C22.2, C25.2, C27.2, C30.2, C36.2, C69.2, J5.10 (Pin_10), J5.12 (Pin_12), J5.14 (Pin_14), J5.16 (Pin_16), J5.18 (Pin_18), J5.2 (Pin_2), J5.20 (Pin_20), J5.22 (Pin_22), J5.24 (Pin_24), J5.4 (Pin_4), J5.6 (Pin_6), J5.8 (Pin_8), U3.4 (VSS), U3.9 (EP)
- net H723_RX: now also J5.23 (Pin_23)
- net H723_TX: now also J5.21 (Pin_21)
- net PSSI_D0: now also J5.1 (Pin_1)
- net PSSI_D1: now also J5.3 (Pin_3)
- net PSSI_D2: now also J5.5 (Pin_5)
- net PSSI_D3: now also J5.7 (Pin_7)
- net PSSI_D4: now also J5.9 (Pin_9)
- net PSSI_D5: now also J5.11 (Pin_11)
- net PSSI_D6: now also J5.13 (Pin_13)
- net PSSI_D7: now also J5.15 (Pin_15)
- net PSSI_DE: now also J5.19 (Pin_19)
- net PSSI_PDCK: now also J5.17 (Pin_17)
- net ULPI_CK: now also R5.2; no longer U4.14 (CLKOUT)
- net VBUS: now also C16.2, C69.1, R29.1, R30.2; no longer U1.8 (VBUS)
- net at U1.1 (VDD): now also R30.1
- net at C35.1, U4.15 (VDD1.8), U4.26 (VDD1.8): now also C36.1
- net at U4.4 (VBUS): now also R3.2
- net QSPI_IO3: now reaches U2.23 (PA1)
- net QSPI_IO3: now also U3.7 (SIO)
- net QSPI_IO0: now reaches U2.24 (PA2)
- net QSPI_IO0: now also U3.5 (SI/SIO)
- net QSPI_IO2: now reaches U2.31 (PA7)
- net QSPI_IO2: now also U3.3 (SIO)
- net QSPI_CLK: now reaches U2.36 (PB2)
- net QSPI_CLK: now also U3.6 (SCLK)
- net QSPI_IO1: now reaches U2.59 (PD12)
- net QSPI_IO1: now also U3.2 (SO/SIO)
- net FMC_A18: no longer names the net of U2.60 (PD13)
- net FMC_D0: no longer names the net of U2.61 (PD14)
- net FMC_D1: no longer names the net of U2.62 (PD15)
- net FMC_D10: no longer names the net of U2.43 (PE13)
- net FMC_D11: no longer names the net of U2.44 (PE14)
- net FMC_D12: no longer names the net of U2.45 (PE15)
- net FMC_D13: no longer names the net of U2.55 (PD8)
- net FMC_D14: no longer names the net of U2.56 (PD9)
- net FMC_D15: no longer names the net of U2.57 (PD10)
- net FMC_D2: no longer names the net of U2.81 (PD0)
- net FMC_D3: no longer names the net of U2.82 (PD1)
- net FMC_D4: no longer names the net of U2.37 (PE7)
- net FMC_D5: no longer names the net of U2.38 (PE8)
- net FMC_D6: no longer names the net of U2.39 (PE9)
- net FMC_D7: no longer names the net of U2.40 (PE10)
- net FMC_D8 renamed QSPI_NCS
- net QSPI_NCS: now also U3.1 (/CE)
- net FMC_D9: no longer names the net of U2.42 (PE12)
- net FMC_NE1: no longer names the net of U2.88 (PD7)
- net FMC_NOE: no longer names the net of U2.85 (PD4)
- net FMC_NWE: no longer names the net of U2.86 (PD5)
- net ULPI_RST: no longer names the net of U4.9 (RESET)
- new net: R5.1, U4.14 (CLKOUT)
- new net: FB3.2, J6.2 (Pin_2)
- new net: R29.2, U1.8 (VBUS)
- new net +5V: C27.1, C30.1, R3.1
- no-connect marks 13 -> 10
Other:
- sheet PowerManagement ports: added 5V; removed none
- note added: "Display Connectors"
- note added: "PSRAM Chip"
- note removed: "Display Connector"
- note removed: "GPIO Input"
- note removed: "GPIO Output"
- moved on the sheet: C15, C19, C20, C21, FB2, J6, R1, U1, Y1

Commit message: layout
Parts:
- added J7: Conn_01x06_Socket, Connector_JST:JST_PH_S6B-PH-K_1x06_P2.00mm_Horizontal, symbol Connector:Conn_01x06_Socket
- added J8: Conn_01x02_Socket, Connector_JST:JST_PH_S2B-PH-K_1x02_P2.00mm_Horizontal, symbol Connector:Conn_01x02_Socket
- added J9: Conn_01x03_Socket, Connector_JST:JST_PH_S3B-PH-K_1x03_P2.00mm_Horizontal, symbol Connector:Conn_01x03_Socket
Connections:
- net +3.3V: now also J8.1 (Pin_1)
- net GND: now also J7.6 (Pin_6), J8.2 (Pin_2), J9.2 (Pin_2)
- new net FGEN_MOSI: J7.1 (Pin_1)
- new net FGEN_SAMP: J7.3 (Pin_3)
- new net FGEN_SCLK: J7.2 (Pin_2)
- new net FGEN_SGAIN: J7.4 (Pin_4)
- new net FGEN_SOFF: J7.5 (Pin_5)
- new net OP_AMP+: J9.1 (Pin_1)
- new net OP_AMP-: J9.3 (Pin_3)
Other:
- note added: "Function Generator Data Connector"
- note added: "Function Generator Op Amp Power"
- note added: "Function Generator Power"
- moved on the sheet: J3

Commit message: 2026-01-11
Parts:
- removed FB3: 100R@100MHz, Inductor_SMD:L_0805_2012Metric, symbol Device:FerriteBead
- removed J2: Conn_01x05_Socket, Connector_JST:JST_PH_S5B-PH-K_1x05_P2.00mm_Horizontal, symbol Connector:Conn_01x05_Socket
- removed J3, J8: Conn_01x02_Socket, Connector_JST:JST_PH_S2B-PH-K_1x02_P2.00mm_Horizontal, symbol Connector:Conn_01x02_Socket
- removed J4: Conn_01x08_Socket, Connector_JST:JST_PH_S8B-PH-K_1x08_P2.00mm_Horizontal, symbol Connector:Conn_01x08_Socket
- removed J5: Conn_02x12_Odd_Even, Connector_JST:JST_PUD_S24B-PUDSS-1_2x12_P2.00mm_Horizontal, symbol Connector_Generic:Conn_02x12_Odd_Even
- removed J6, J9: Conn_01x03_Socket, Connector_JST:JST_PH_S3B-PH-K_1x03_P2.00mm_Horizontal, symbol Connector:Conn_01x03_Socket
- removed J7: Conn_01x06_Socket, Connector_JST:JST_PH_S6B-PH-K_1x06_P2.00mm_Horizontal, symbol Connector:Conn_01x06_Socket
- added D10, D11, D12, D13, D14, D15, D4, D5, D6, D7, D8, D9: LED, LED_SMD:LED_0805_2012Metric, symbol Device:LED
- added F1, F10, F11, F12, F2, F3, F4, F5, F6, F7, F8, F9: 500MA/24V, Fuse:Fuse_1206_3216Metric, symbol JLC_PARTS:500MA/24V
- added H1, H2, H3, H4: MountingHole_Pad, MountingHole:MountingHole_3.2mm_M3_Pad_Via, symbol Mechanical:MountingHole_Pad
- added R32, R37, R40, R43: 330R, Resistor_SMD:R_0603_1608Metric, symbol Device:R
- added R33, R34, R35, R36, R38, R39, R41, R42: 2.2K, Resistor_SMD:R_0603_1608Metric, symbol Device:R
- added U10: FFC2B28-24-G, JLC_PARTS:FPC-SMD_24P-P0.50_XKB_X05A10L24G, symbol JLC_PARTS:FFC2B28-24-G
- added U11: SM08B-PASS-TBT(LF)(SN), JLC_PARTS:CONN-SMD_SM08B-PASS-TBT-LF-SN, symbol JLC_PARTS:SM08B-PASS-TBT(LF)(SN)
- added U12, U15, U16, U17: SM05B-PASS-TBT(LF)(SN), JLC_PARTS:CONN-SMD_5P-P2.00_SM05B-PASS-TBT-LF-SN, symbol JLC_PARTS:SM05B-PASS-TBT(LF)(SN)
- added U13: SM02B-PASS-TBT(LF)(SN), JLC_PARTS:CONN-SMD_SM02B-PASS-TBT, symbol JLC_PARTS:SM02B-PASS-TBT(LF)(SN)
- added U14: SM06B-PASS-TBT(LF)(SN), JLC_PARTS:CONN-SMD_SM06B-PASS-TBT, symbol JLC_PARTS:SM06B-PASS-TBT(LF)(SN)
- added U9: S5B-ZR-SM4A-TF(LF)(SN), JLC_PARTS:CONN-SMD_5P-P1.50_S5B-ZR-SM4A-TF-LF-SN, symbol JLC_PARTS:S5B-ZR-SM4A-TF(LF)(SN)
Connections:
- net +3.3V: now also F1.1, F10.1, F4.1, F7.1, U11.1, U11.8, U9.4
- net DISP_DC: now also U11.6
- net DISP_MOSI: now also U11.3
- net DISP_NSS: now also U11.5
- net DISP_RST: now also U11.7
- net DISP_SCK: now also U11.4
- net FGEN_MOSI: now also U14.1
- net FGEN_SAMP: now also U14.3
- net FGEN_SCLK: now also U14.2
- net FGEN_SGAIN: now also U14.4
- net FGEN_SOFF: now also U14.5
- net GND: now also D10.2 (A), D11.1 (K), D12.1 (K), D13.2 (A), D14.1 (K), D15.1 (K), D4.2 (A), D5.1 (K), D6.1 (K), D7.2 (A), D8.1 (K), D9.1 (K), H1.1, H2.1, H3.1, H4.1, U10.10, U10.12, U10.14, U10.16, U10.18, U10.2, U10.20, U10.22, U10.25, U10.26, U10.4, U10.6, U10.8, U11.10, U11.2, U11.9, U12.2, U12.3, U12.6, U12.7, U13.2, U13.3, U13.4, U14.6, U14.7, U14.8, U15.2, U15.3, U15.6, U15.7, U16.2, U16.3, U16.6, U16.7, U17.2, U17.3, U17.6, U17.7, U9.2, U9.6, U9.7
- net H723_RX: now also U2.97 (PE0), U10.23
- net H723_TX: now also U2.98 (PE1), U10.24
- net OP_AMP+: now also F11.1, F2.1, F5.1, F8.1
- net OP_AMP-: now also F12.1, F3.1, F6.1, F9.1
- net PSSI_D0: now also U10.1
- net PSSI_D1: now also U10.3
- net PSSI_D2: now also U10.5
- net PSSI_D3: now also U10.7
- net PSSI_D4: now also U2.79 (PC11), U10.13; no longer U2.3 (PE4)
- net PSSI_D5: now also U10.15
- net PSSI_D6: now also U2.95 (PB8), U10.19; no longer U2.4 (PE5)
- net PSSI_D7: now also U2.96 (PB9), U10.21; no longer U2.5 (PE6)
- net PSSI_DE: now also U10.11
- net PSSI_PDCK: now also U10.9
- net PSSI_RDY: now also U10.17
- net SWCLK: now also U9.5
- net SWDIO: now also U9.3
- net V_SELECT: now also U13.1
- net nRST: now also U9.1
- new net: D15.2 (A), R43.2
- new net: F8.2, R42.1, U17.4
- new net: F3.2, R35.1, U15.5
- new net: D7.1 (K), R35.2
- new net: F4.2, R40.1, U16.1
- new net: F5.2, R39.1, U16.4
- new net: F6.2, R38.1, U16.5
- new net: F1.2, R37.1, U15.1
- new net: D14.2 (A), R42.2
- new net: D12.2 (A), R40.2
- new net: F2.2, R36.1, U15.4
- new net: F7.2, R43.1, U17.1
- new net: F9.2, R41.1, U17.5
- new net: D8.2 (A), R36.2
- new net: D4.1 (K), R34.2
- new net: F10.2, R32.1, U12.1
- new net: D6.2 (A), R32.2
- new net: F11.2, R33.1, U12.4
- new net: D5.2 (A), R33.2
- new net: D9.2 (A), R37.2
- new net: F12.2, R34.1, U12.5
- new net: D11.2 (A), R39.2
- new net: D13.1 (K), R41.2
- new net: D10.1 (K), R38.2
Other:
- note added: "Mounting Holes"
- note added: "Oscilloscope Board Data Connector"
- note added: "Power Connector"
- note added: "Variable Power Supply Connector"
- note removed: "Function Generator Op Amp Power"
- note removed: "Function Generator Power"
- note removed: "Oscilloscope Board Connectors"
- note removed: "Variable PSU Power Connector"
- moved on the sheet: C22, C23, C24, C25, C26, C27, C28, C29, C30, C31, C32, C33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
Changed lines of the file:
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@@
 	(generator "eeschema")
 	(generator_version "9.0")
-	(paper "A3")
+	(paper "A2")

Commit message: new layout
Parts:
- removed D10, D11, D12, D13, D14, D15, D4, D5, D6, D7, D8, D9: LED, LED_SMD:LED_0805_2012Metric, symbol Device:LED
- removed F1, F10, F11, F12, F2, F3, F4, F5, F6, F7, F8, F9: 500MA/24V, Fuse:Fuse_1206_3216Metric, symbol JLC_PARTS:500MA/24V
- removed R32, R37, R40, R43: 330R, Resistor_SMD:R_0603_1608Metric, symbol Device:R
- removed R33, R34, R35, R36, R38, R39, R41, R42: 2.2K, Resistor_SMD:R_0603_1608Metric, symbol Device:R
- added U18, U19, U21: SM05B-PASS-TBT(LF)(SN), JLC_PARTS:CONN-SMD_5P-P2.00_SM05B-PASS-TBT-LF-SN, symbol JLC_PARTS:SM05B-PASS-TBT(LF)(SN)
- added U20: SM08B-PASS-TBT(LF)(SN), JLC_PARTS:CONN-SMD_SM08B-PASS-TBT-LF-SN, symbol JLC_PARTS:SM08B-PASS-TBT(LF)(SN)
- C34, C35: footprint Capacitor_SMD:C_0603_1608Metric -> Capacitor_SMD:C_0402_1005Metric
Connections:
- net +3.3V: now also U12.1, U15.1, U16.1, U17.1, U18.1, U19.1
- net DISP_DC: now also U2.82 (PD1)
- net DISP_MOSI: now also U2.80 (PC12)
- net DISP_NSS: no longer U11.5
- net DISP_RST: now also U2.83 (PD2)
- net DISP_SCK: now also U2.78 (PC10)
- net FGEN_MOSI: now also U2.88 (PD7)
- net FGEN_SAMP: now also U2.90 (PB4(NJTRST))
- net FGEN_SCLK: now also U2.89 (PB3(JTDO)
- net FGEN_SGAIN: now also U2.92 (PB6)
- net FGEN_SOFF: now also U2.1 (PE2)
- net GND: now also U18.2, U18.3, U18.6, U18.7, U19.2, U19.3, U19.6, U19.7, U20.10, U20.3, U20.9, U21.1, U21.6, U21.7
- net OP_AMP+: now also U12.4, U15.4, U16.4, U17.4, U18.4, U19.4
- net OP_AMP-: now also U12.5, U15.5, U16.5, U17.5, U18.5, U19.5
- net ADC1_INP4: now reaches U2.32 (PC4)
- net ADC1_INP4: now also U20.1
- net ADC2_INP8: now reaches U2.33 (PC5)
- net ADC2_INP8: now also U20.2
- net R_SRC_1K: now reaches U2.37 (PE7)
- net R_SRC_1K: now also U20.4
- net R_SRC_100K: now reaches U2.38 (PE8)
- net R_SRC_100K: now also U20.5
- net V_RANGE_LOW: now reaches U2.39 (PE9)
- net V_RANGE_LOW: now also U20.6
- net V_RANGE_HIGH: now reaches U2.40 (PE10)
- net V_RANGE_HIGH: now also U20.7
- net BUZZER_CTRL: now reaches U2.43 (PE13)
- net BUZZER_CTRL: now also U20.8
- net SPI2_MISO: now reaches U2.53 (PB14)
- net SPI2_MISO: now also U21.3
- net SPI2_MOSI: now reaches U2.54 (PB15)
- net SPI2_MOSI: now also U21.4
- net SPI2_CS: now reaches U2.55 (PD8)
- net SPI2_CS: now also U21.5
- net SPI2_CK: now reaches U2.68 (PA9)
- net SPI2_CK: now also U21.2
- net DISP_CS: now reaches U2.81 (PD0)
- net DISP_CS: now also U11.5
- net USB_C_PG: no longer names the net of U1.10 (PG)
Other:
- note added: "Logic Analyzer"
- note added: "Multimeter GPIO"
- moved on the sheet: U12, U15, U16, U17

Commit message: updated connectors
Parts:
- removed U20: SM08B-PASS-TBT(LF)(SN), JLC_PARTS:CONN-SMD_SM08B-PASS-TBT-LF-SN, symbol JLC_PARTS:SM08B-PASS-TBT(LF)(SN)
- removed U21: SM05B-PASS-TBT(LF)(SN), JLC_PARTS:CONN-SMD_5P-P2.00_SM05B-PASS-TBT-LF-SN, symbol JLC_PARTS:SM05B-PASS-TBT(LF)(SN)
- added U20: SM06B-PASS-TBT(LF)(SN), JLC_PARTS:CONN-SMD_SM06B-PASS-TBT, symbol JLC_PARTS:SM06B-PASS-TBT(LF)(SN)
- added U22: SM09B-PASS-TBT(LF)(SN), JLC_PARTS:CONN-SMD_SM09B-PASS-TBT, symbol JLC_PARTS:SM09B-PASS-TBT(LF)(SN)
Connections:
- net ADC1_INP4: now also U22.1
- net ADC2_INP8: now also U22.2
- net BUZZER_CTRL: now also U22.9
- net GND: now also U20.1, U20.7, U20.8, U22.10, U22.11, U22.3
- net R_SRC_100K: now also U22.5
- net R_SRC_1K: now also U22.4
- net SPI2_CK: now also U20.2
- net SPI2_CS: now also U20.5
- net SPI2_MISO: now also U20.3
- net SPI2_MOSI: now also U20.4
- net V_RANGE_HIGH: now also U22.7
- net V_RANGE_LOW: now also U22.6
- net MULT_CONN_IND: now reaches U2.42 (PE12)
- net MULT_CONN_IND: now also U22.8
- net LOGAN_CONN_IND: now reaches U2.56 (PD9)
- net LOGAN_CONN_IND: now also U20.6
