File: Electrical/MainBoard/DebuggingBoard.kicad_sch (KiCad schematic)
At the start: 72 parts, among them J1 Barrel_Jack_Switch, SW1 SW_SPDT, U1 CH224K, U10 FFC2B28-24-G, U11 SM08B-PASS-TBT(LF)(SN), U12 SM05B-PASS-TBT(LF)(SN), U13 SM02B-PASS-TBT(LF)(SN), U14 SM06B-PASS-TBT(LF)(SN), U15 SM05B-PASS-TBT(LF)(SN), U16 SM05B-PASS-TBT(LF)(SN), U17 SM05B-PASS-TBT(LF)(SN), U18 SM05B-PASS-TBT(LF)(SN), U19 SM05B-PASS-TBT(LF)(SN), U2 STM32H723VGTx, U20 SM06B-PASS-TBT(LF)(SN), U22 SM09B-PASS-TBT(LF)(SN), U3 APS6404L-3SQR-ZR, U4 USB3300-EZK, U9 S5B-ZR-SM4A-TF(LF)(SN), Y1 X322525MOB4SI, Y2 X322524MOB4SI

Commit message: vpsu conn
Parts:
- added U21: SM06B-PASS-TBT(LF)(SN), JLC_Parts:CONN-SMD_SM06B-PASS-TBT, symbol JLC_PARTS:SM06B-PASS-TBT(LF)(SN)
Connections:
- net GND: now also U21.4
- net V_POS_I: now reaches U2.44 (PE14)
- net V_POS_I: now also U21.2
- net V_NEG_I: now reaches U2.45 (PE15)
- net V_NEG_I: now also U21.3
- new net VPSU_CONN_IND: U21.1

Commit message: finished main
Parts:
- removed U14: SM06B-PASS-TBT(LF)(SN), JLC_PARTS:CONN-SMD_SM06B-PASS-TBT, symbol JLC_PARTS:SM06B-PASS-TBT(LF)(SN)
- removed U18, U19: SM05B-PASS-TBT(LF)(SN), JLC_PARTS:CONN-SMD_5P-P2.00_SM05B-PASS-TBT-LF-SN, symbol JLC_PARTS:SM05B-PASS-TBT(LF)(SN)
- added C57, C58: 100nF, Capacitor_SMD:C_0402_1005Metric, symbol Device:C
- added D1, D4, D5: LED, LED_SMD:LED_0603_1608Metric, symbol Device:LED
- added R22: 10K, Resistor_SMD:R_0402_1005Metric, symbol Device:R
- added R25, R34, R35: 1K, Resistor_SMD:R_0402_1005Metric, symbol Device:R
- added R32, R33: 4.7K, Resistor_SMD:R_0402_1005Metric, symbol Device:R
- added TP10, TP11, TP6, TP7, TP8, TP9: TestPoint, TestPoint:TestPoint_Pad_D2.5mm, symbol Connector:TestPoint
- added U14: SM08B-PASS-TBT(LF)(SN), JLC_PARTS:CONN-SMD_SM08B-PASS-TBT-LF-SN, symbol JLC_PARTS:SM08B-PASS-TBT(LF)(SN)
- added U18, U19: SM03B-PASS-TBT(LF)(SN)_C412099, JLC_PARTS:CONN-SMD_SM03B-PASS-TBT, symbol JLC_PARTS:SM03B-PASS-TBT(LF)(SN)_C412099
- added U23: SM05B-PASS-TBT(LF)(SN), JLC_PARTS:CONN-SMD_5P-P2.00_SM05B-PASS-TBT-LF-SN, symbol JLC_PARTS:SM05B-PASS-TBT(LF)(SN)
- added U24: SM04B-PASS-TBT(LF)(SN), JLC_PARTS:CONN-SMD_SM04B-PASS-TBT-LF-SN, symbol JLC_PARTS:SM04B-PASS-TBT(LF)(SN)
- added U26: SM06B-PASS-TBT(LF)(SN), JLC_PARTS:CONN-SMD_SM06B-PASS-TBT, symbol JLC_PARTS:SM06B-PASS-TBT(LF)(SN)
- U21: footprint JLC_Parts:CONN-SMD_SM06B-PASS-TBT -> JLC_PARTS:CONN-SMD_SM06B-PASS-TBT
Connections:
- net +3.3V: now also R22.1, TP7.1, U18.1, U19.1, U26.2
- net +3.3VA: now also TP11.1
- net +5V: now also TP8.1, U18.3, U19.3
- net BOOT0: now also TP10.1
- net DISP_CS: now also U2.85 (PD4); no longer U2.81 (PD0)
- net DISP_DC: now also U2.86 (PD5); no longer U2.82 (PD1)
- net DISP_RST: now also U2.87 (PD6); no longer U2.83 (PD2)
- net FGEN_MOSI: now also U14.1
- net FGEN_SAMP: now also U14.4
- net FGEN_SCLK: now also U14.2
- net FGEN_SGAIN: now also U14.5
- net FGEN_SOFF: now also U2.2 (PE3), U14.6; no longer U2.1 (PE2)
- net GND: now also U21.3, U21.7, U21.8, C57.2, C58.2, D1.1 (K), D4.1 (K), D5.1 (K), U14.10, U14.3, U14.9, U18.2, U18.4, U18.5, U19.2, U19.4, U19.5, U23.3, U23.6, U23.7, U24.4, U24.5, U24.6, U26.3, U26.7, U26.8; no longer U21.4
- net USB_PD_PG: now also U1.10 (PG), U2.57 (PD10), R22.2
- net VBUS: now also TP6.1
- net VPSU_CONN_IND: now also U2.9 (PC15), U21.4; no longer U21.1
- net V_NEG_I: now also U2.16 (PC1), U21.6; no longer U2.45 (PE15), U21.3
- net V_POS_I: now also U2.22 (PA0), U21.5; no longer U2.44 (PE14), U21.2
- net nRST: now also TP9.1
- net GPIO: now reaches U2.3 (PE4)
- net GPIO: now also U14.8
- net at U2.4 (PE5): now also R32.2
- net at U2.5 (PE6): now also R33.2
- net BUTTON: now reaches U2.58 (PD11)
- net BUTTON: now also U26.1
- net ENC_A: now reaches U2.60 (PD13)
- net ENC_A: now also U26.4
- net ENC_B: now reaches U2.61 (PD14)
- net ENC_B: now also U26.5
- net ENC_BUTTON: now reaches U2.62 (PD15)
- net ENC_BUTTON: now also U26.6
- net LED2: now reaches U2.69 (PA10)
- net LED2: now also R35.1
- net COMP_RST: now reaches U2.7 (PC13)
- net COMP_RST: now also U23.5
- net CAN_RX: now reaches U2.70 (PA11)
- net CAN_RX: now also U24.2
- net CAN_TX: now reaches U2.71 (PA12)
- net CAN_TX: now also U24.3
- net COMP_CONN_IND: now reaches U2.77 (PA15(JTDI))
- net COMP_CONN_IND: now also U23.4
- net POWER_IND: now reaches U2.8 (PC14)
- new net: D5.2 (A), R35.2
- new net: D1.2 (A), R25.2
- new net: D4.2 (A), R34.2
- new net CAN_CONN_IND: U2.83 (PD2), U24.1
- new net DBUG_LED: R25.1, U2.44 (PE14)
- new net FGEN_CONN_IND: U14.7, U2.1 (PE2)
- new net LED3: R34.1, U2.45 (PE15)
- new net UART4_RX: U2.81 (PD0), U23.2
- new net UART4_TX: U2.82 (PD1), U23.1
- new net V_NEG_DAC: C57.1, R33.1, U21.2
- new net V_POS_DAC: C58.1, R32.1, U21.1
Other:
- sheet PowerManagement ports: added POWER_IND; removed none
- note added: "CAN Transciever Board"
- note added: "Component Tester Board"
- note added: "Interface Board"
- note added: "VPSU Data Connector"
- note removed: "Unconnected GPIO"
- moved on the sheet: C3, C8, H1, H2, H3, H4, U10, U11, U12, U13, U15, U16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

Commit message: manufactured
Parts:
- removed TP8: TestPoint, TestPoint:TestPoint_Pad_D2.5mm, symbol Connector:TestPoint
- added TP1: TestPoint, TestPoint:TestPoint_Pad_D2.0mm, symbol Connector:TestPoint
- TP10, TP11, TP6, TP7, TP9: footprint TestPoint:TestPoint_Pad_D2.5mm -> TestPoint:TestPoint_Pad_D2.0mm
Connections:
- net GND: now also TP1.1
