File: Electrical/MainBoard/DebuggingBoard.kicad_pcb (KiCad board)
At the start: 6 copper layers, 120 x 80 mm, 132 parts, among them J1 Barrel_Jack_Switch, J2 Conn_01x05_Socket, J3 Conn_01x02_Socket, J4 Conn_01x08_Socket, J5 Conn_02x12_Odd_Even, J6 Conn_01x03_Socket, Q1 AO3401A, SW1 SW_SPDT, U1 CH224K, U2 STM32H723VGTx, U3 APS6404L-3SQR-ZR, U4 USB3300-EZK, U5 TPS65131RGE, U6 TPS2121RUXR, U7 TPS7A9401DSCR, U8 LM61460AASQRJRRQ1, Y1 X322525MOB4SI, Y2 X322524MOB4SI

Commit message: layout main
Parts:
- added C70: 10uF, Capacitor_SMD:C_0603_1608Metric, F.Cu at (173.9, 86.9)
- added C71: 22uF, Capacitor_SMD:C_0805_2012Metric, F.Cu at (176.2, 79.7)
- added C72: 22uF, Capacitor_SMD:C_0805_2012Metric, F.Cu at (163.2, 79.7)
- added R31: 100K, Resistor_SMD:R_0402_1005Metric, F.Cu at (184.4, 84.0)
- C64, C67: value 47uF -> 22uF
- R10, R17, R18, R7, R8, R9: footprint Resistor_SMD:R_0402_1005Metric -> Resistor_SMD:R_0603_1608Metric
- R12: value 12.4K -> 10K; footprint Resistor_SMD:R_0603_1608Metric -> Resistor_SMD:R_0402_1005Metric
- R13: value 187K -> 150K
- R23: value 100K -> 33K
- R26: value 100K -> 30K; footprint Resistor_SMD:R_0402_1005Metric -> Resistor_SMD:R_0603_1608Metric
- R27: value 24.9K -> 7.5K
- R6: footprint Resistor_SMD:R_0603_1608Metric -> Resistor_SMD:R_0402_1005Metric
- moved C34 151.5 mm to (241.4, 97.3)
- moved C35 147.3 mm to (235.4, 86.5), turned to 180 degrees
- moved C13 141.0 mm to (225.0, 84.0), turned to 90 degrees
- moved R2 135.0 mm to (247.8, 112.8), turned to -90 degrees
- moved C9 134.5 mm to (220.9, 100.0)
- moved C48 131.4 mm to (193.6, 83.6), turned to -90 degrees
- moved C56 129.7 mm to (197.1, 79.0), turned to -90 degrees
- moved C36 129.1 mm to (235.4, 95.6), turned to -90 degrees
- moved C40 126.5 mm to (188.0, 78.3)
- moved C59 125.8 mm to (202.0, 78.9), turned to -90 degrees
- moved C51 123.5 mm to (191.1, 78.3), turned to 180 degrees
- moved R21 122.3 mm to (192.2, 83.3), turned to -90 degrees
- moved C37 121.7 mm to (184.2, 76.6)
- moved C61 119.8 mm to (203.1, 78.9), turned to -90 degrees
- moved U7 119.5 mm to (189.6, 82.3)
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Connections:
- U7 pad 4: GND -> Net-(U7-PG)
Routing:
- net /ULPI_D4: track 41.1 -> 49.6 mm
- net /ULPI_DIR: track 41.0 -> 49.5 mm
- net /ULPI_D6: track 41.0 -> 49.5 mm
- net /ULPI_D3: track 41.1 -> 49.6 mm
- net /ULPI_D5: track 41.0 -> 49.5 mm
- net /ULPI_CK: track 41.0 -> 49.4 mm
- net /ULPI_D7: track 40.8 -> 49.2 mm
- net /ULPI_NXT: track 41.1 -> 49.5 mm
- net /ULPI_STP: track 41.0 -> 49.4 mm
- net /ULPI_D2: track 41.0 -> 49.4 mm
- net /ULPI_D0: track 41.2 -> 49.5 mm
- net /ULPI_D1: track 41.0 -> 49.2 mm
- net Net-(U6-OV1): track 0.00 -> 8.08 mm
- net +3.3V: track 0.00 -> 6.69 mm
- net Net-(U2-VDDA): track 0.00 -> 5.35 mm
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
Commit message: layout
Parts:
- removed FB3: 100R@100MHz, Inductor_SMD:L_0805_2012Metric
- added J7: Conn_01x06_Socket, Connector_JST:JST_PH_S6B-PH-K_1x06_P2.00mm_Horizontal, F.Cu at (183.7, 58.6)
- added J8: Conn_01x02_Socket, Connector_JST:JST_PH_S2B-PH-K_1x02_P2.00mm_Horizontal, F.Cu at (168.7, 58.6)
- added J9: Conn_01x03_Socket, Connector_JST:JST_PH_S3B-PH-K_1x03_P2.00mm_Horizontal, F.Cu at (161.6, 58.6)
- J6: value Conn_01x03_Socket -> Conn_01x02_Socket; footprint Connector_JST:JST_PH_S3B-PH-K_1x03_P2.00mm_Horizontal -> Connector_JST:JST_PH_S2B-PH-K_1x02_P2.00mm_Horizontal
- moved R2 50.2 mm to (247.3, 62.7)
- moved SW1 50.2 mm to (252.6, 63.1)
- moved J3 20.8 mm to (190.7, 58.6)
- moved J6 18.5 mm to (197.7, 58.6)
- moved J4 18.1 mm to (216.7, 58.6)
- moved J5 17.4 mm to (243.3, 62.7)
- moved C60 1.60 mm to (168.7, 89.8)
- moved C63 1.60 mm to (172.6, 85.5)
- moved C64 1.60 mm to (174.1, 78.1)
- moved C65 1.60 mm to (165.4, 85.4)
- moved C67 1.60 mm to (165.3, 78.1)
- moved C70 1.60 mm to (173.9, 85.3)
- moved C71 1.60 mm to (176.2, 78.1)
- moved C72 1.60 mm to (163.2, 78.1)
- moved R22 1.60 mm to (173.1, 91.8)
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Connections:
- net /PowerManagement/OP_AMP+ renamed /OP_AMP+
- net /PowerManagement/OP_AMP- renamed /OP_AMP-
- J6 pad 2: Net-(J6-Pin_2) -> GND

Commit message: 2026-01-11
Parts:
- removed J2: Conn_01x05_Socket, Connector_JST:JST_PH_S5B-PH-K_1x05_P2.00mm_Horizontal
- removed J3, J6, J8: Conn_01x02_Socket, Connector_JST:JST_PH_S2B-PH-K_1x02_P2.00mm_Horizontal
- removed J4: Conn_01x08_Socket, Connector_JST:JST_PH_S8B-PH-K_1x08_P2.00mm_Horizontal
- removed J5: Conn_02x12_Odd_Even, Connector_JST:JST_PUD_S24B-PUDSS-1_2x12_P2.00mm_Horizontal
- removed J7: Conn_01x06_Socket, Connector_JST:JST_PH_S6B-PH-K_1x06_P2.00mm_Horizontal
- removed J9: Conn_01x03_Socket, Connector_JST:JST_PH_S3B-PH-K_1x03_P2.00mm_Horizontal
- added D10: LED, LED_SMD:LED_0805_2012Metric, F.Cu at (158.5, 65.4)
- added D11: LED, LED_SMD:LED_0805_2012Metric, F.Cu at (154.5, 65.5)
- added D12: LED, LED_SMD:LED_0805_2012Metric, F.Cu at (150.5, 65.5)
- added D13: LED, LED_SMD:LED_0805_2012Metric, F.Cu at (154.5, 73.9)
- added D14: LED, LED_SMD:LED_0805_2012Metric, F.Cu at (150.5, 73.9)
- added D15: LED, LED_SMD:LED_0805_2012Metric, F.Cu at (158.5, 73.9)
- added D4: LED, LED_SMD:LED_0805_2012Metric, F.Cu at (158.5, 91.1)
- added D5: LED, LED_SMD:LED_0805_2012Metric, F.Cu at (150.5, 91.0)
- added D6: LED, LED_SMD:LED_0805_2012Metric, F.Cu at (154.5, 90.9)
- added D7: LED, LED_SMD:LED_0805_2012Metric, F.Cu at (158.5, 81.4)
- added D8: LED, LED_SMD:LED_0805_2012Metric, F.Cu at (150.5, 81.4)
- added D9: LED, LED_SMD:LED_0805_2012Metric, F.Cu at (154.5, 81.4)
- added F1: 500MA/24V, Fuse:Fuse_1206_3216Metric, F.Cu at (166.1, 67.1)
- added F10: 500MA/24V, Fuse:Fuse_1206_3216Metric, F.Cu at (166.1, 79.5)
- added F11: 500MA/24V, Fuse:Fuse_1206_3216Metric, F.Cu at (166.1, 87.0)
- added F12: 500MA/24V, Fuse:Fuse_1206_3216Metric, F.Cu at (166.1, 92.0)
- added F2: 500MA/24V, Fuse:Fuse_1206_3216Metric, F.Cu at (166.1, 72.0)
- added F3: 500MA/24V, Fuse:Fuse_1206_3216Metric, F.Cu at (166.1, 77.0)
- added F4: 500MA/24V, Fuse:Fuse_1206_3216Metric, F.Cu at (166.1, 74.5)
- added F5: 500MA/24V, Fuse:Fuse_1206_3216Metric, F.Cu at (166.1, 69.5)
- added F6: 500MA/24V, Fuse:Fuse_1206_3216Metric, F.Cu at (166.1, 64.7)
- added F7: 500MA/24V, Fuse:Fuse_1206_3216Metric, F.Cu at (166.1, 89.5)
- added F8: 500MA/24V, Fuse:Fuse_1206_3216Metric, F.Cu at (166.1, 84.5)
- added F9: 500MA/24V, Fuse:Fuse_1206_3216Metric, F.Cu at (166.1, 82.0)
- added H1: MountingHole_Pad, MountingHole:MountingHole_3.2mm_M3_Pad_Via, F.Cu at (142.0, 57.5)
- added H2: MountingHole_Pad, MountingHole:MountingHole_3.2mm_M3_Pad_Via, F.Cu at (142.0, 122.5)
- added H3: MountingHole_Pad, MountingHole:MountingHole_3.2mm_M3_Pad_Via, F.Cu at (247.5, 122.5)
- added H4: MountingHole_Pad, MountingHole:MountingHole_3.2mm_M3_Pad_Via, F.Cu at (247.5, 57.5)
- added R32: 330R, Resistor_SMD:R_0603_1608Metric, F.Cu at (152.5, 90.8)
- added R33: 2.2K, Resistor_SMD:R_0603_1608Metric, F.Cu at (148.5, 90.8)
- added R34: 2.2K, Resistor_SMD:R_0603_1608Metric, F.Cu at (156.5, 90.8)
- added R35: 2.2K, Resistor_SMD:R_0603_1608Metric, F.Cu at (156.5, 81.5)
- added R36: 2.2K, Resistor_SMD:R_0603_1608Metric, F.Cu at (148.5, 81.3)
- added R37: 330R, Resistor_SMD:R_0603_1608Metric, F.Cu at (152.5, 81.3)
- added R38: 2.2K, Resistor_SMD:R_0603_1608Metric, F.Cu at (156.5, 65.2)
- added R39: 2.2K, Resistor_SMD:R_0603_1608Metric, F.Cu at (152.5, 65.3)
- added R40: 330R, Resistor_SMD:R_0603_1608Metric, F.Cu at (148.5, 65.3)
- added R41: 2.2K, Resistor_SMD:R_0603_1608Metric, F.Cu at (152.5, 73.8)
- added R42: 2.2K, Resistor_SMD:R_0603_1608Metric, F.Cu at (148.5, 73.8)
- added R43: 330R, Resistor_SMD:R_0603_1608Metric, F.Cu at (156.5, 73.8)
- added U10: FFC2B28-24-G, JLC_PARTS:FPC-SMD_24P-P0.50_XKB_X05A10L24G, F.Cu at (235.5, 52.0)
- added U11: SM08B-PASS-TBT(LF)(SN), JLC_PARTS:CONN-SMD_SM08B-PASS-TBT-LF-SN, F.Cu at (217.5, 56.9)
- added U12: SM05B-PASS-TBT(LF)(SN), JLC_PARTS:CONN-SMD_5P-P2.00_SM05B-PASS-TBT-LF-SN, F.Cu at (142.5, 86.3)
- added U13: SM02B-PASS-TBT(LF)(SN), JLC_PARTS:CONN-SMD_SM02B-PASS-TBT, F.Cu at (142.8, 98.6)
- added U14: SM06B-PASS-TBT(LF)(SN), JLC_PARTS:CONN-SMD_SM06B-PASS-TBT, F.Cu at (198.5, 57.0)
- added U15: SM05B-PASS-TBT(LF)(SN), JLC_PARTS:CONN-SMD_5P-P2.00_SM05B-PASS-TBT-LF-SN, B.Cu at (142.5, 86.3)
- added U16: SM05B-PASS-TBT(LF)(SN), JLC_PARTS:CONN-SMD_5P-P2.00_SM05B-PASS-TBT-LF-SN, B.Cu at (142.5, 70.8)
- added U17: SM05B-PASS-TBT(LF)(SN), JLC_PARTS:CONN-SMD_5P-P2.00_SM05B-PASS-TBT-LF-SN, F.Cu at (142.5, 70.8)
- added U9: S5B-ZR-SM4A-TF(LF)(SN), JLC_PARTS:CONN-SMD_5P-P1.50_S5B-ZR-SM4A-TF-LF-SN, F.Cu at (251.2, 78.7)
- moved C54 58.6 mm to (159.0, 120.5)
- moved C55 58.6 mm to (165.0, 119.5)
- moved C57 58.6 mm to (159.0, 119.5)
- moved C58 58.6 mm to (165.0, 120.5)
- moved FB5 58.6 mm to (158.5, 123.0)
- moved FB7 58.6 mm to (164.5, 122.9)
- moved C45 37.7 mm to (177.6, 66.9)
- moved C46 37.7 mm to (179.1, 66.1)
- moved D3 37.7 mm to (185.9, 65.7)
- moved R6 37.7 mm to (183.9, 74.0)
- moved C47 37.7 mm to (181.8, 66.6)
- moved C53 37.7 mm to (181.3, 63.8)
- moved C38 37.7 mm to (183.3, 75.3)
- moved C39 37.7 mm to (182.3, 73.5)
- moved C41 37.7 mm to (181.0, 76.1)
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Connections:
- U2 pad 3: /PSSI_D4 -> unconnected-(U2-PE4-Pad3)
- U2 pad 4: /PSSI_D6 -> unconnected-(U2-PE5-Pad4)
- U2 pad 5: /PSSI_D7 -> unconnected-(U2-PE6-Pad5)
- U2 pad 79: unconnected-(U2-PC11-Pad79) -> /PSSI_D4
- U2 pad 95: unconnected-(U2-PB8-Pad95) -> /PSSI_D6
- U2 pad 96: unconnected-(U2-PB9-Pad96) -> /PSSI_D7
- U2 pad 97: unconnected-(U2-PE0-Pad97) -> /H723_RX
- U2 pad 98: unconnected-(U2-PE1-Pad98) -> /H723_TX
Routing:
- net /PSSI_D2: track 0.00 -> 61.1 mm
- net /PSSI_D0: track 0.00 -> 61.1 mm
- net /PSSI_D1: track 0.00 -> 61.1 mm
- net /PSSI_D3: track 0.00 -> 61.1 mm
- net /PSSI_RDY: track 0.00 -> 61.0 mm
- net /PSSI_D4: track 0.00 -> 61.0 mm
- net /PSSI_D6: track 0.00 -> 61.0 mm
- net /PSSI_D7: track 0.00 -> 61.0 mm
- net /PSSI_D5: track 0.00 -> 61.0 mm
- net /PSSI_DE: track 0.00 -> 59.9 mm, vias 0 -> 2
- net /PSSI_PDCK: track 0.00 -> 59.9 mm, vias 0 -> 2
- net /BOOT0: track 0.00 -> 41.6 mm, vias 0 -> 2
- net /H723_RX: track 0.00 -> 37.3 mm
- net /H723_TX: track 0.00 -> 37.3 mm
- net /QSPI_NCS: track 24.1 -> 18.0 mm
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Other:
- outline, holes or cut-outs redrawn
- board text added: "+12V"
- board text added: "-12V"
- board text added: "3.3V"

Commit message: new layout
Parts:
- removed C57, C58: 10nF, Capacitor_SMD:C_0402_1005Metric
- removed D10, D11, D12, D13, D14, D15, D4, D5, D6, D7, D8, D9: LED, LED_SMD:LED_0805_2012Metric
- removed F1, F10, F11, F12, F2, F3, F4, F5, F6, F7, F8, F9: 500MA/24V, Fuse:Fuse_1206_3216Metric
- removed FB5, FB7: 600R@100MHz, Inductor_SMD:L_0805_2012Metric
- removed R32, R37, R40, R43: 330R, Resistor_SMD:R_0603_1608Metric
- removed R33, R34, R35, R36, R38, R39, R41, R42: 2.2K, Resistor_SMD:R_0603_1608Metric
- added U18: SM05B-PASS-TBT(LF)(SN), JLC_PARTS:CONN-SMD_5P-P2.00_SM05B-PASS-TBT-LF-SN, F.Cu at (77.6, 63.8)
- added U19: SM05B-PASS-TBT(LF)(SN), JLC_PARTS:CONN-SMD_5P-P2.00_SM05B-PASS-TBT-LF-SN, B.Cu at (77.6, 63.9)
- added U20: SM08B-PASS-TBT(LF)(SN), JLC_PARTS:CONN-SMD_SM08B-PASS-TBT-LF-SN, F.Cu at (121.9, 128.1)
- added U21: SM05B-PASS-TBT(LF)(SN), JLC_PARTS:CONN-SMD_5P-P2.00_SM05B-PASS-TBT-LF-SN, F.Cu at (140.1, 127.6)
- C34, C35: footprint Capacitor_SMD:C_0603_1608Metric -> Capacitor_SMD:C_0402_1005Metric
- C54, C55: value 100nF -> 1uF; footprint Capacitor_SMD:C_0402_1005Metric -> Capacitor_SMD:C_0603_1608Metric
- moved R2 104.6 mm to (150.9, 109.0)
- moved U9 102.7 mm to (156.0, 117.3)
- moved SW1 102.3 mm to (157.6, 105.5)
- moved R7 100.0 mm to (89.6, 122.3), turned to -90 degrees
- moved R24 98.6 mm to (86.0, 113.6), turned to 90 degrees
- moved C70 98.6 mm to (86.2, 116.2), turned to 90 degrees
- moved R25 98.5 mm to (86.0, 111.6), turned to 90 degrees
- moved R10 98.3 mm to (91.2, 122.3), turned to 90 degrees
- moved R8 97.2 mm to (89.6, 125.4), turned to -90 degrees
- moved R4 97.2 mm to (148.2, 95.6), turned to -90 degrees
- moved R22 96.3 mm to (87.1, 109.6), turned to 90 degrees
- moved R23 96.3 mm to (87.1, 111.6), turned to 90 degrees
- moved R1 95.9 mm to (148.0, 103.6), turned to -90 degrees
- moved C63 95.8 mm to (87.6, 115.9), turned to 90 degrees
- moved R9 95.4 mm to (91.2, 125.4), turned to 90 degrees
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Connections:
- C47 pad 2: Net-(D3-A) -> /OP_AMP-
- C50 pad 1: Net-(D2-K) -> /OP_AMP+
- C52 pad 1: Net-(D2-K) -> /OP_AMP+
- C53 pad 1: Net-(D3-A) -> /OP_AMP-
- D2 pad 1: Net-(D2-K) -> /OP_AMP+
- D3 pad 2: Net-(D3-A) -> /OP_AMP-
- R16 pad 1: Net-(D2-K) -> /OP_AMP+
- R19 pad 1: Net-(D3-A) -> /OP_AMP-
- U1 pad 10: /USB_C_PG -> unconnected-(U1-PG-Pad10)
- U11 pad 5: /DISP_NSS -> /DISP_CS
- U12 pad 1: Net-(F10-Pad2) -> +3.3V
- U12 pad 4: Net-(F11-Pad2) -> /OP_AMP+
- U12 pad 5: Net-(F12-Pad2) -> /OP_AMP-
- U15 pad 1: Net-(F1-Pad2) -> +3.3V
- U15 pad 4: Net-(F2-Pad2) -> /OP_AMP+
- U15 pad 5: Net-(F3-Pad2) -> /OP_AMP-
- U16 pad 1: Net-(F4-Pad2) -> +3.3V
- U16 pad 4: Net-(F5-Pad2) -> /OP_AMP+
- U16 pad 5: Net-(F6-Pad2) -> /OP_AMP-
- U17 pad 1: Net-(F7-Pad2) -> +3.3V
- U17 pad 4: Net-(F8-Pad2) -> /OP_AMP+
- U17 pad 5: Net-(F9-Pad2) -> /OP_AMP-
- U2 pad 1: unconnected-(U2-PE2-Pad1) -> /FGEN_SOFF
- U2 pad 32: unconnected-(U2-PC4-Pad32) -> /ADC1_INP4
- U2 pad 33: unconnected-(U2-PC5-Pad33) -> /ADC2_INP8
- U2 pad 37: unconnected-(U2-PE7-Pad37) -> /R_SRC_1K
- U2 pad 38: unconnected-(U2-PE8-Pad38) -> /R_SRC_100K
- U2 pad 39: unconnected-(U2-PE9-Pad39) -> /V_RANGE_LOW
- U2 pad 40: unconnected-(U2-PE10-Pad40) -> /V_RANGE_HIGH
- U2 pad 43: unconnected-(U2-PE13-Pad43) -> /BUZZER_CTRL
- U2 pad 53: unconnected-(U2-PB14-Pad53) -> /SPI2_MISO
- U2 pad 54: unconnected-(U2-PB15-Pad54) -> /SPI2_MOSI
- U2 pad 55: unconnected-(U2-PD8-Pad55) -> /SPI2_CS
- U2 pad 68: unconnected-(U2-PA9-Pad68) -> /SPI2_CK
- U2 pad 78: unconnected-(U2-PC10-Pad78) -> /DISP_SCK
- U2 pad 80: unconnected-(U2-PC12-Pad80) -> /DISP_MOSI
- U2 pad 81: unconnected-(U2-PD0-Pad81) -> /DISP_CS
- U2 pad 82: unconnected-(U2-PD1-Pad82) -> /DISP_DC
- U2 pad 83: unconnected-(U2-PD2-Pad83) -> /DISP_RST
- U2 pad 88: unconnected-(U2-PD7-Pad88) -> /FGEN_MOSI
- U2 pad 89: unconnected-(U2-PB3(JTDO-Pad89) -> /FGEN_SCLK
- U2 pad 90: unconnected-(U2-PB4(NJTRST)-Pad90) -> /FGEN_SAMP
- U2 pad 92: unconnected-(U2-PB6-Pad92) -> /FGEN_SGAIN
- U5 pad 15: Net-(D3-A) -> /OP_AMP-
- U5 pad 23: Net-(D2-K) -> /OP_AMP+
Routing:
- net /nRST: track 1.96 -> 50.3 mm, vias 0 -> 2
- net /SWDIO: track 0.00 -> 43.9 mm, vias 0 -> 2
- net /SWCLK: track 0.00 -> 41.9 mm, vias 0 -> 2
- net /SPI2_CK: track 0.00 -> 41.7 mm, vias 0 -> 2
- net /SPI2_CS: track 0.00 -> 37.3 mm
- net /SPI2_MOSI: track 0.00 -> 35.9 mm
- net /ADC2_INP8: track 0.00 -> 35.8 mm, vias 0 -> 2
- net /SPI2_MISO: track 0.00 -> 34.3 mm
- net /ADC1_INP4: track 0.00 -> 32.2 mm, vias 0 -> 2
- net /FGEN_SOFF: track 0.00 -> 31.8 mm, vias 0 -> 2
- net /R_SRC_1K: track 0.00 -> 31.6 mm
- net /R_SRC_100K: track 0.00 -> 31.1 mm
- net /ULPI_D7: track 49.3 -> 18.7 mm
- net /V_RANGE_LOW: track 0.00 -> 30.5 mm
- net /V_RANGE_HIGH: track 0.00 -> 29.9 mm
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- added copper zone on F.Cu, net +3.3V
- removed copper zone on In2.Cu, net GND
Other:
- board size 120 x 80 mm -> 89.9 x 90 mm
- board text removed: "+12V"
- board text removed: "-12V"
- board text removed: "3.3V"

Commit message: updated connectors
Parts:
- removed U21: SM05B-PASS-TBT(LF)(SN), JLC_PARTS:CONN-SMD_5P-P2.00_SM05B-PASS-TBT-LF-SN
- added U22: SM09B-PASS-TBT(LF)(SN), JLC_PARTS:CONN-SMD_SM09B-PASS-TBT, F.Cu at (119.1, 128.2)
- U20: value SM08B-PASS-TBT(LF)(SN) -> SM06B-PASS-TBT(LF)(SN); footprint JLC_PARTS:CONN-SMD_SM08B-PASS-TBT-LF-SN -> JLC_PARTS:CONN-SMD_SM06B-PASS-TBT
- moved U20 17.3 mm to (139.2, 128.2)
- moved C10 0.12 mm to (133.5, 99.3)
- moved C9 0.10 mm to (132.9, 100.6)
Connections:
- U2 pad 42: unconnected-(U2-PE12-Pad42) -> /MULT_CONN_IND
- U2 pad 56: unconnected-(U2-PD9-Pad56) -> /LOGAN_CONN_IND
- U20 pad 1: /ADC1_INP4 -> GND
- U20 pad 2: /ADC2_INP8 -> /SPI2_CK
- U20 pad 3: GND -> /SPI2_MISO
- U20 pad 4: /R_SRC_1K -> /SPI2_MOSI
- U20 pad 5: /R_SRC_100K -> /SPI2_CS
- U20 pad 6: /V_RANGE_LOW -> /LOGAN_CONN_IND
- U20 pad 7: /V_RANGE_HIGH -> GND
- U20 pad 8: /BUZZER_CTRL -> GND
Routing:
- net /LOGAN_CONN_IND: track 0.00 -> 38.9 mm
- net /MULT_CONN_IND: track 0.00 -> 29.7 mm
- net /R_SRC_1K: track 31.6 -> 32.4 mm
- net /ADC2_INP8: track 35.8 -> 36.6 mm
- net /ADC1_INP4: track 32.2 -> 33.0 mm
- net /V_RANGE_LOW: track 30.5 -> 31.2 mm
- net /V_RANGE_HIGH: track 29.9 -> 30.6 mm
- net /R_SRC_100K: track 31.1 -> 31.8 mm
- net /SPI2_MISO: track 34.3 -> 34.9 mm

Commit message: vpsu conn
Routing:
- net /ADC2_INP8: track 36.6 -> 37.4 mm
- net /ADC1_INP4: track 33.0 -> 33.8 mm
- net /BUZZER_CTRL: track 29.0 -> 29.7 mm
- net /MULT_CONN_IND: track 29.7 -> 30.3 mm
- net /R_SRC_100K: track 31.8 -> 32.4 mm
- net /R_SRC_1K: track 32.4 -> 33.0 mm
- net /V_RANGE_LOW: track 31.2 -> 31.8 mm
- net /V_RANGE_HIGH: track 30.6 -> 31.2 mm

Commit message: finished main
Parts:
- added C57: 100nF, Capacitor_SMD:C_0402_1005Metric, F.Cu at (115.7, 85.5)
- added C58: 100nF, Capacitor_SMD:C_0402_1005Metric, F.Cu at (115.7, 83.5)
- added D4: LED, LED_SMD:LED_0603_1608Metric, F.Cu at (158.2, 60.9)
- added D5: LED, LED_SMD:LED_0603_1608Metric, F.Cu at (158.2, 56.4)
- added R32: 4.7K, Resistor_SMD:R_0402_1005Metric, F.Cu at (117.2, 83.9)
- added R33: 4.7K, Resistor_SMD:R_0402_1005Metric, F.Cu at (117.2, 85.0)
- added R34: 1K, Resistor_SMD:R_0402_1005Metric, F.Cu at (156.0, 61.0)
- added R35: 1K, Resistor_SMD:R_0402_1005Metric, F.Cu at (156.0, 56.6)
- added TP1: TestPoint, TestPoint:TestPoint_Pad_D2.5mm, F.Cu at (31.7, 98.5)
- added TP10: TestPoint, TestPoint:TestPoint_Pad_D2.5mm, F.Cu at (112.8, 76.3)
- added TP11: TestPoint, TestPoint:TestPoint_Pad_D2.5mm, F.Cu at (47.4, 103.0)
- added TP2: TestPoint, TestPoint:TestPoint_Pad_D2.5mm, F.Cu at (31.7, 103.0)
- added TP3: TestPoint, TestPoint:TestPoint_Pad_D2.5mm, F.Cu at (31.7, 107.6)
- added TP4: TestPoint, TestPoint:TestPoint_Pad_D2.5mm, F.Cu at (31.7, 112.2)
- added TP5: TestPoint, TestPoint:TestPoint_Pad_D2.5mm, F.Cu at (31.7, 116.7)
- added TP6: TestPoint, TestPoint:TestPoint_Pad_D2.5mm, F.Cu at (38.2, 98.5)
- added TP7: TestPoint, TestPoint:TestPoint_Pad_D2.5mm, F.Cu at (38.2, 103.0)
- added TP8: TestPoint, TestPoint:TestPoint_Pad_D2.5mm, F.Cu at (42.8, 98.5)
- added TP9: TestPoint, TestPoint:TestPoint_Pad_D2.5mm, F.Cu at (42.8, 103.0)
- added U21: SM06B-PASS-TBT(LF)(SN), JLC_PARTS:CONN-SMD_SM06B-PASS-TBT, F.Cu at (90.0, 127.8)
- added U23: SM05B-PASS-TBT(LF)(SN), JLC_PARTS:CONN-SMD_5P-P2.00_SM05B-PASS-TBT-LF-SN, F.Cu at (90.4, 52.4)
- added U24: SM04B-PASS-TBT(LF)(SN), JLC_PARTS:CONN-SMD_SM04B-PASS-TBT-LF-SN, F.Cu at (126.0, 52.3)
- added U26: SM06B-PASS-TBT(LF)(SN), JLC_PARTS:CONN-SMD_SM06B-PASS-TBT, F.Cu at (152.9, 105.3)
- FB4: value 600R@100MHz -> 120R@100MHz; footprint Inductor_SMD:L_0805_2012Metric -> Inductor_SMD:L_0603_1608Metric
- FB6: value 100R@100MHz -> 120R@100MHz; footprint Inductor_SMD:L_0805_2012Metric -> Inductor_SMD:L_0603_1608Metric
- R11: footprint Resistor_SMD:R_0402_1005Metric -> Resistor_SMD:R_0603_1608Metric
- R14: value 1K -> 10K
- R22: value 100K -> 10K
- R25: value 47.5K -> 1K
- U14: value SM06B-PASS-TBT(LF)(SN) -> SM08B-PASS-TBT(LF)(SN); footprint JLC_PARTS:CONN-SMD_SM06B-PASS-TBT -> JLC_PARTS:CONN-SMD_SM08B-PASS-TBT-LF-SN
- U18, U19: value SM05B-PASS-TBT(LF)(SN) -> SM03B-PASS-TBT(LF)(SN)_C412099; footprint JLC_PARTS:CONN-SMD_5P-P2.00_SM05B-PASS-TBT-LF-SN -> JLC_PARTS:CONN-SMD_SM03B-PASS-TBT
- moved D1 90.9 mm to (158.2, 58.6), turned to 180 degrees
- moved R25 87.7 mm to (156.0, 58.8)
- moved R22 58.3 mm to (145.3, 112.8), turned to 180 degrees
- moved SW1 30.1 mm to (144.6, 132.7), turned to 0 degrees
- moved R2 19.7 mm to (144.1, 127.5), turned to 0 degrees
- moved C42 18.4 mm to (104.6, 114.2)
- moved R10 18.1 mm to (101.0, 107.1)
- moved R17 18.1 mm to (105.6, 110.2)
- moved R18 18.1 mm to (105.6, 107.1)
- moved R7 18.1 mm to (99.4, 107.1)
- moved R8 18.1 mm to (99.4, 110.2)
- moved R9 18.1 mm to (101.0, 110.2)
- moved U6 18.1 mm to (103.2, 111.8)
- moved R11 17.8 mm to (102.9, 115.2)
- moved U14 15.9 mm to (108.5, 51.8)
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Connections:
- D1 pad 1: Net-(D1-K) -> GND
- R14 pad 1: /V_SELECT -> +3.3V
- R14 pad 2: Net-(D1-A) -> /POWER_IND
- R22 pad 1: Net-(U8-PGOOD) -> +3.3V
- R22 pad 2: +5V -> /USB_PD_PG
- R25 pad 1: Net-(U8-EN/SYNC) -> /DBUG_LED
- R25 pad 2: GND -> Net-(D1-A)
- U1 pad 10: unconnected-(U1-PG-Pad10) -> /USB_PD_PG
- U14 pad 3: /FGEN_SAMP -> GND
- U14 pad 4: /FGEN_SGAIN -> /FGEN_SAMP
- U14 pad 5: /FGEN_SOFF -> /FGEN_SGAIN
- U14 pad 6: GND -> /FGEN_SOFF
- U14 pad 7: GND -> /FGEN_CONN_IND
- U14 pad 8: GND -> /GPIO
- U18 pad 3: GND -> +5V
- U18 pad 4: /OP_AMP+ -> GND
- U18 pad 5: /OP_AMP- -> GND
- U19 pad 3: GND -> +5V
- U19 pad 4: /OP_AMP+ -> GND
- U19 pad 5: /OP_AMP- -> GND
- U2 pad 1: /FGEN_SOFF -> /FGEN_CONN_IND
- U2 pad 16: unconnected-(U2-PC1-Pad16) -> /V_NEG_I
- U2 pad 2: unconnected-(U2-PE3-Pad2) -> /FGEN_SOFF
- U2 pad 22: unconnected-(U2-PA0-Pad22) -> /V_POS_I
- U2 pad 3: unconnected-(U2-PE4-Pad3) -> /GPIO
- U2 pad 4: unconnected-(U2-PE5-Pad4) -> Net-(U2-PE5)
- U2 pad 44: unconnected-(U2-PE14-Pad44) -> /DBUG_LED
- U2 pad 45: unconnected-(U2-PE15-Pad45) -> /LED3
- U2 pad 5: unconnected-(U2-PE6-Pad5) -> Net-(U2-PE6)
- U2 pad 57: unconnected-(U2-PD10-Pad57) -> /USB_PD_PG
- U2 pad 58: unconnected-(U2-PD11-Pad58) -> /BUTTON
- U2 pad 60: unconnected-(U2-PD13-Pad60) -> /ENC_A
- U2 pad 61: unconnected-(U2-PD14-Pad61) -> /ENC_B
- U2 pad 62: unconnected-(U2-PD15-Pad62) -> /ENC_BUTTON
- U2 pad 69: unconnected-(U2-PA10-Pad69) -> /LED2
- U2 pad 7: unconnected-(U2-PC13-Pad7) -> /COMP_RST
- U2 pad 70: unconnected-(U2-PA11-Pad70) -> /CAN_RX
- U2 pad 71: unconnected-(U2-PA12-Pad71) -> /CAN_TX
- U2 pad 77: unconnected-(U2-PA15(JTDI)-Pad77) -> /COMP_CONN_IND
- U2 pad 8: unconnected-(U2-PC14-Pad8) -> /POWER_IND
- U2 pad 81: /DISP_CS -> /UART4_RX
- U2 pad 82: /DISP_DC -> /UART4_TX
- U2 pad 83: /DISP_RST -> /CAN_CONN_IND
- U2 pad 85: unconnected-(U2-PD4-Pad85) -> /DISP_CS
- U2 pad 86: unconnected-(U2-PD5-Pad86) -> /DISP_DC
- U2 pad 87: unconnected-(U2-PD6-Pad87) -> /DISP_RST
- U2 pad 9: unconnected-(U2-PC15-Pad9) -> /VPSU_CONN_IND
- U6 pad 9: Net-(D1-K) -> /POWER_IND
- U8 pad 5: Net-(U8-PGOOD) -> unconnected-(U8-PGOOD-Pad5)
Routing:
- net +3.3V: track 23.2 -> 176.2 mm, vias 0 -> 26
- net +5V: track 3.21 -> 108.7 mm, vias 0 -> 41
- net /COMP_CONN_IND: track 0.00 -> 69.4 mm, vias 0 -> 2
- net /V_POS_DAC: track 0.00 -> 63.5 mm, vias 0 -> 2
- net /UART4_RX: track 0.00 -> 63.4 mm, vias 0 -> 2
- net /VPSU_CONN_IND: track 0.00 -> 61.4 mm, vias 0 -> 2
- net /V_NEG_DAC: track 0.00 -> 60.8 mm, vias 0 -> 2
- net /UART4_TX: track 0.00 -> 60.1 mm, vias 0 -> 2
- net /COMP_RST: track 0.00 -> 58.9 mm, vias 0 -> 2
- net /LED2: track 0.00 -> 57.0 mm, vias 0 -> 2
- net /V_NEG_I: track 0.00 -> 53.0 mm, vias 0 -> 2
- net /DBUG_LED: track 0.00 -> 52.7 mm, vias 0 -> 2
- net /POWER_IND: track 0.00 -> 52.1 mm, vias 0 -> 2
- net /V_POS_I: track 0.00 -> 50.7 mm, vias 0 -> 2
- net /LED3: track 0.00 -> 50.3 mm, vias 0 -> 2
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- added copper zone on F.Cu, net +12V
- added copper zone on In3.Cu, net +12V
- added copper zone on In3.Cu, net +3.3V
- added copper zone on F.Cu, net +3.3VA
- added copper zone on In3.Cu, net +3.3VA
- added copper zone on F.Cu, net +5V
- added copper zone on In3.Cu, net +5V
- added copper zone on F.Cu, net /OP_AMP+
- added copper zone on In3.Cu, net /OP_AMP+
- added copper zone on F.Cu, net /OP_AMP-
- added copper zone on In3.Cu, net /OP_AMP-
- added copper zone on F.Cu, net /V_SELECT
- added copper zone on In3.Cu, net /V_SELECT
- added copper zone on F.Cu, net Net-(D2-A)
- added copper zone on F.Cu, net Net-(D3-K)
- added copper zone on F.Cu, net Net-(Q1-D)
- added copper zone on F.Cu, net Net-(U5-ENN)
- added copper zone on F.Cu, net Net-(U7-EN_UV)
- added copper zone on F.Cu, net Net-(U7-SNS)
- added copper zone on F.Cu, net Net-(U8-CBOOT)
- added copper zone on F.Cu, net Net-(U8-SW)
- added copper zone on F.Cu, net VBUS
- added copper zone on In3.Cu, net VBUS
Other:
- board size 89.9 x 90 mm -> 90 x 90 mm
- board text added: "+-12V/GND/3.3V"
- board text added: "3.3V/5V/GND"
- board text added: "BOOT0 1/0"
- board text added: "CANBUS DEBUGGER"
- board text added: "COMPONENT TESTER"
- board text added: "DISPLAY"
- board text added: "FUNCTION GEN"
- board text added: "INTERFACE"
- board text added: "LOGIC ANALYZER"
- board text added: "MULTIMETER"
- board text added: "OSCILLOSCOPE"
- board text added: "SWD"
- board text added: "VPSU"
- board text added: "VPSU PWR"
