File: Electrical/MainBoard/DebuggingBoard.kicad_pcb (KiCad board)
At the start: 6 copper layers, 90 x 90 mm, 166 parts, among them J1 Barrel_Jack_Switch, Q1 AO3401A, SW1 SW_SPDT, U1 CH224K, U10 FFC2B28-24-G, U11 SM08B-PASS-TBT(LF)(SN), U12 SM05B-PASS-TBT(LF)(SN), U13 SM02B-PASS-TBT(LF)(SN), U14 SM08B-PASS-TBT(LF)(SN), U15 SM05B-PASS-TBT(LF)(SN)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

Commit message: manufactured
Parts:
- removed TP8: TestPoint, TestPoint:TestPoint_Pad_D2.5mm
- added G***: LOGO, LOGO, F.Cu at (117.9, 69.8)
- added U25: PJ-002BH, JLC_PARTS:DC-IN-TH_PJ-002BH, F.Cu at (78.9, 120.0)
- TP1, TP10, TP11, TP2, TP3, TP4, TP5, TP6, TP7, TP9: footprint TestPoint:TestPoint_Pad_D2.5mm -> TestPoint:TestPoint_Pad_D2.0mm
- moved TP9 106.8 mm to (148.1, 121.0)
- moved TP6 102.3 mm to (139.9, 110.4)
- moved TP4 93.6 mm to (110.1, 61.0)
- moved TP1 76.5 mm to (108.2, 99.0)
- moved TP3 73.5 mm to (88.5, 61.0)
- moved TP2 66.2 mm to (97.8, 99.0)
- moved TP5 65.8 mm to (97.5, 115.4)
- moved TP11 61.8 mm to (108.1, 91.6)
- moved TP7 60.6 mm to (97.8, 91.6)
- moved TP10 36.7 mm to (137.9, 103.0)
- moved U18 0.47 mm to (76.7, 63.3)
- moved U19 0.47 mm to (76.7, 63.3)
- moved U13 0.30 mm to (77.0, 106.8)
- moved U24 0.20 mm to (126.0, 52.1)
- moved U17 0.20 mm to (77.3, 77.2)
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Connections:
- TP1 pad 1: /POWER_IND -> GND
Routing:
- net /OP_AMP-: track 26.6 -> 39.5 mm
- net /OP_AMP+: track 9.08 -> 16.6 mm, vias 8 -> 9
- net VBUS: track 8.48 -> 13.5 mm
- net /V_SELECT: track 9.54 -> 14.2 mm
- net /BOOT0: track 57.3 -> 60.0 mm, vias 2 -> 3
- net +3.3V: track 176.2 -> 178.2 mm, vias 26 -> 27
- net +5V: track 108.7 -> 108.4 mm, vias 41 -> 42
- net GND: vias 106 -> 108
- net +3.3VA: vias 8 -> 9
Other:
- board text added: "+12V"
- board text added: "-12V"
- board text added: "3.3V"
- board text added: "3.3VA"
- board text added: "5V"
- board text added: "BOOT0"
- board text added: "BOOT0 I/O"
- board text added: "GND"
- board text added: "MAIN BOARD"
- board text added: "NRST"
- board text added: "SHARKBYTE DEBUGGER"
- board text added: "SYSTEM V"
- board text added: "VBUS"
- board text added: "±12V/GND/3.3V"
- board text removed: "+-12V/GND/3.3V"
- board text removed: "BOOT0 1/0"

Commit message: software unit testing
Parts:
- removed U25: PJ-002BH, JLC_PARTS:DC-IN-TH_PJ-002BH
Connections:
- C66 pad 2: +5V -> Net-(U8-SW)
