File: Electrical/MainBoard/PowerManagement.kicad_sch (KiCad schematic)
At the start: 79 parts, among them Q1 AO3401A, Q2 AO3401A, U2 AP62300TWU, U3 TPS65131RGE, U4 TPS2121RUXR, U5 TPS7A9401DSCR, U7 LM393, U8 AMS1117-3.3

Commit message: VPSU schem complete
Parts:
- removed C14, C43, C51, C53: 10uF, symbol Device:C
- removed C15, C16: 22uF, symbol Device:C
- removed C17, C48, C50, C52: 100nF, symbol Device:C
- removed D4: SS34, Diode_SMD:D_SMA, symbol Diode:SS34
- removed FB5: 100R@100MHz, symbol Device:FerriteBead
- removed FB6: 600R@100MHz, symbol Device:FerriteBead
- removed L1: FNR6045S4R7, symbol Device:L
- removed Q1: AO3401A, Rocketry_Easyeda:SOT-23_L2.9-W1.3-P1.90-LS2.4-BR, symbol ROCKETRY_EASYEDA:AO3401A
- removed Q2: AO3401A, Rocketry_Easyeda:SOT-23_L2.9-W1.3-P1.90-LS2.4-BR, symbol Rocketry_Easyeda:AO3401A
- removed R1: 13K, symbol Device:R
- removed R10: 33K, symbol Device:R
- removed R2: 20K, symbol Device:R
- removed R4: 60.4K, symbol Device:R
- removed R5: 10K, symbol Device:R
- removed U2: AP62300TWU, Package_TO_SOT_SMD:TSOT-23-6, symbol Regulator_Switching:AP62300TWU
- removed U7: LM393, symbol Comparator:LM393
- removed U8: AMS1117-3.3, Rocketry_Easyeda:SOT-223-3_L6.5-W3.4-P2.30-LS7.0-BR, symbol Rocketry_Easyeda:AMS1117-3.3
- added C18, C21: 100nF, symbol Device:C
- added C27: 1uF, symbol Device:C
- added C38, C46: 47uF, symbol Device:C
- added C39: 10uF, symbol Device:C
- added C47: 22pF, symbol Device:C
- added L2: FNR6045S4R7, symbol Device:L
- added Q1: AO3401A, Rocketry_Easyeda:SOT-23_L2.9-W1.3-P1.90-LS2.4-BR, symbol Rocketry_Easyeda:AO3401A
- added R13: 24.9K, symbol Device:R
- added R14: 1K, symbol Device:R
- added R25, R26, R6: 100K, symbol Device:R
- added R27: 47.5K, symbol Device:R
- added U9: LM61460AASQRJRRQ1, Rocketry_Easyeda:VQFN-14-HR_L4.0-W3.5-TL_LM61460AASQRJRRQ1, symbol Rocketry_Easyeda:LM61460AASQRJRRQ1
- C34: value 10uF -> 100nF
- R17: renamed from R13; value 10K -> 33K
- R19: renamed from R8; value 10K -> 27K
- renumbered C30 to C19, C19 to C20, C20 to C22, C31 to C23, C21 to C24, C32 to C25, C27 to C26, C24 to C29, C25 to C30, C33 to C31, C36 to C32, C22 to C33, C23 to C36, C26 to C37, C39 to C40, C40 to C42, C42 to C43, C37 to C44, C38 to C45, C18 to C48, D2 to D1, D3 to D2, D1 to D4, FB1 to FB2, FB7 to FB3, FB3 to FB5, FB2 to FB6, L2 to L1, R20 to R10, R18 to R11, R22 to R12, R7 to R15, R6 to R16, R14 to R18, R15 to R20, R11 to R21, R12 to R22, R16 to R3, R24 to R4, R23 to R5, R19 to R7, R17 to R8, U3 to U4, U4 to U8
Connections:
- net +5V: now also C34.2, R9.1, C38.1, C46.1, L2.2, Q1.2 (S), R14.1, R25.2, U9.1 (BIAS)
- net 3.3V: now also C35.1; no longer C34.1
- net 3.3VA: now also FB6.2
- net GND: now also U8.3 (CP2), C18.1, C21.2, C27.2, C38.2, C39.2, C46.2, R13.2, R27.2, R6.2, U9.11 (PGND2), U9.3 (AGND), U9.9 (PGND1); no longer C34.2
- net VBUS: no longer R9.1
- net V_SELECT: now also C18.2, C21.1, R26.1, U9.12 (VIN2), U9.8 (VIN1)
- net at C24.1, L1.1: now also Q1.3 (D)
- net at C32.1, FB3.1, R5.2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: now also C39.1; no longer C35.1
- net at R9.2: now also C47.2, R13.1, U9.4 (FB); no longer U8.3 (CP2)
- net at U4.7 (BSW): now also Q1.1 (G)
- new net: R26.2, R27.1, U9.7 (EN/SYNC)
- new net: L2.1, U9.10 (SW)
- new net: C47.1, R14.2
- new net: R25.1, U9.5 (PGOOD)
- new net: C27.1, U9.2 (VCC)
- new net: C34.1, U9.13 (RBOOT), U9.14 (CBOOT)
- new net: R6.1, U9.6 (RT)
Other:
- note added: "High-Current High-Duty 5V Buck"
- note removed: "12V Buck to 5.136V"
- note removed: "5.37V"
- note removed: "Comparator Power"
- note removed: "If 12V, 12*(13/33) = 4.73V > 3.3V (Pulled High) But if 5V, 5*(13/33) = 1.97V < 3.3V (Pulled Low)"
- note removed: "Unused Comparator"
- note removed: "Voltage Buck Bypass if at 5V"
- moved on the sheet: C20, C22, C24, C26, C28, C29, C30, C33, C36, C37, C40, C41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

Commit message: layout
Parts:
- C37: renamed from C19; footprint (none) -> Capacitor_SMD:C_0603_1608Metric
- C38: renamed from C20; footprint (none) -> Capacitor_SMD:C_0603_1608Metric
- C39: renamed from C22; footprint (none) -> Capacitor_SMD:C_0402_1005Metric
- C40: renamed from C23; footprint (none) -> Capacitor_SMD:C_0603_1608Metric
- C41: renamed from C24; footprint (none) -> Capacitor_SMD:C_0603_1608Metric
- C42: renamed from C48; footprint (none) -> Capacitor_SMD:C_0402_1005Metric
- C43: renamed from C25; footprint (none) -> Capacitor_SMD:C_0402_1005Metric
- C44: renamed from C26; footprint (none) -> Capacitor_SMD:C_0402_1005Metric
- C45: renamed from C28; footprint (none) -> Capacitor_SMD:C_0402_1005Metric
- C46: renamed from C29; footprint (none) -> Capacitor_SMD:C_0402_1005Metric
- C47: renamed from C30; footprint (none) -> Capacitor_SMD:C_0402_1005Metric
- C48: renamed from C31; footprint (none) -> Capacitor_SMD:C_0603_1608Metric
- C49: renamed from C32; footprint (none) -> Capacitor_SMD:C_0402_1005Metric
- C50: renamed from C33; footprint (none) -> Capacitor_SMD:C_0402_1005Metric
- C51: renamed from C39; footprint (none) -> Capacitor_SMD:C_0603_1608Metric
- C52: renamed from C36; footprint (none) -> Capacitor_SMD:C_0805_2012Metric
- C53: renamed from C37; footprint (none) -> Capacitor_SMD:C_0805_2012Metric
- C54: renamed from C40; footprint (none) -> Capacitor_SMD:C_0402_1005Metric
- C55: renamed from C41; footprint (none) -> Capacitor_SMD:C_0402_1005Metric
- C56: renamed from C35; footprint (none) -> Capacitor_SMD:C_0603_1608Metric
- C57: renamed from C42; footprint (none) -> Capacitor_SMD:C_0402_1005Metric
- C58: renamed from C43; footprint (none) -> Capacitor_SMD:C_0402_1005Metric
- C59: renamed from C44; footprint (none) -> Capacitor_SMD:C_0402_1005Metric
- C60: renamed from C27; footprint (none) -> Capacitor_SMD:C_0603_1608Metric
- C61: renamed from C45; footprint (none) -> Capacitor_SMD:C_0402_1005Metric
- C62: renamed from C21; footprint (none) -> Capacitor_SMD:C_0402_1005Metric
- C63: renamed from C18; footprint (none) -> Capacitor_SMD:C_0402_1005Metric
- C64: renamed from C38; footprint (none) -> Capacitor_SMD:C_0805_2012Metric
- C65: renamed from C49; footprint (none) -> Capacitor_SMD:C_0603_1608Metric
- C66: renamed from C34; footprint (none) -> Capacitor_SMD:C_0402_1005Metric
- C67: renamed from C46; footprint (none) -> Capacitor_SMD:C_0805_2012Metric
- C68: renamed from C47; footprint (none) -> Capacitor_SMD:C_0402_1005Metric
- D1: renamed from D4; footprint (none) -> LED_SMD:LED_0603_1608Metric
- FB4: renamed from FB2; footprint (none) -> Inductor_SMD:L_0805_2012Metric
- FB5: renamed from FB4; footprint (none) -> Inductor_SMD:L_0805_2012Metric
- FB6: renamed from FB3; footprint (none) -> Inductor_SMD:L_0805_2012Metric
- FB7: renamed from FB5; footprint (none) -> Inductor_SMD:L_0805_2012Metric
- FB8: renamed from FB6; footprint (none) -> Inductor_SMD:L_0805_2012Metric
- L1: footprint (none) -> Inductor_SMD:L_Changjiang_FNR6045S
- L2: renamed from L3; footprint (none) -> Inductor_SMD:L_Changjiang_FNR6045S
- L3: renamed from L2; footprint (none) -> Inductor_SMD:L_Changjiang_FNR6045S
- R10: renamed from R18; footprint (none) -> Resistor_SMD:R_0402_1005Metric
- R11: renamed from R19; footprint (none) -> Resistor_SMD:R_0402_1005Metric
- R12: renamed from R4; footprint (none) -> Resistor_SMD:R_0603_1608Metric
- R13: renamed from R5; footprint (none) -> Resistor_SMD:R_0603_1608Metric
- R14: renamed from R20; footprint (none) -> Resistor_SMD:R_0402_1005Metric
- R15: renamed from R7; footprint (none) -> Resistor_SMD:R_0402_1005Metric
- R16: renamed from R8; footprint (none) -> Resistor_SMD:R_0402_1005Metric
- R17: renamed from R21; footprint (none) -> Resistor_SMD:R_0402_1005Metric
- R18: renamed from R22; footprint (none) -> Resistor_SMD:R_0402_1005Metric
- R19: renamed from R10; footprint (none) -> Resistor_SMD:R_0402_1005Metric
- R20: renamed from R11; footprint (none) -> Resistor_SMD:R_0402_1005Metric
- R21: renamed from R12; footprint (none) -> Resistor_SMD:R_0402_1005Metric
- R22: renamed from R25; footprint (none) -> Resistor_SMD:R_0402_1005Metric
- R23: renamed from R6; footprint (none) -> Resistor_SMD:R_0402_1005Metric
- R24: renamed from R26; footprint (none) -> Resistor_SMD:R_0402_1005Metric
- R25: renamed from R27; footprint (none) -> Resistor_SMD:R_0402_1005Metric
- R26: renamed from R9; footprint (none) -> Resistor_SMD:R_0402_1005Metric
- R27: renamed from R13; footprint (none) -> Resistor_SMD:R_0603_1608Metric
- R28: renamed from R14; footprint (none) -> Resistor_SMD:R_0402_1005Metric
- R6: renamed from R3; footprint (none) -> Resistor_SMD:R_0603_1608Metric
- R7: renamed from R15; footprint (none) -> Resistor_SMD:R_0402_1005Metric
- R8: renamed from R16; footprint (none) -> Resistor_SMD:R_0402_1005Metric
- R9: renamed from R17; footprint (none) -> Resistor_SMD:R_0402_1005Metric
- renumbered D1 to D2, D2 to D3, U4 to U5, U8 to U6, U5 to U7, U9 to U8

Commit message: layout main
Parts:
- added C70: 10uF, Capacitor_SMD:C_0603_1608Metric, symbol Device:C
- added C71, C72: 22uF, Capacitor_SMD:C_0805_2012Metric, symbol Device:C
- added R31: 100K, Resistor_SMD:R_0402_1005Metric, symbol Device:R
- C64, C67: value 47uF -> 22uF
- R10, R17, R18, R7, R8, R9: footprint Resistor_SMD:R_0402_1005Metric -> Resistor_SMD:R_0603_1608Metric
- R12: value 12.4K -> 10K; footprint Resistor_SMD:R_0603_1608Metric -> Resistor_SMD:R_0402_1005Metric
- R13: value 187K -> 150K
- R23: value 100K -> 33K
- R26: value 100K -> 30K; footprint Resistor_SMD:R_0402_1005Metric -> Resistor_SMD:R_0603_1608Metric
- R27: value 24.9K -> 7.5K
- R6: footprint Resistor_SMD:R_0603_1608Metric -> Resistor_SMD:R_0402_1005Metric
Connections:
- net +5V: now also C71.1, C72.1
- net GND: now also C70.1, C71.2, C72.2; no longer U7.4 (PG)
- net V_SELECT: now also C70.2
- net at C49.1, C51.1, FB6.1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: now also R31.1
- new net: R31.2, U7.4 (PG)
Other:
- moved on the sheet: C38, C39, C41, C44, C45, C46, C47, C50, C52, C53, C54, C55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

Commit message: new layout
Parts:
- removed C57, C58: 10nF, Capacitor_SMD:C_0402_1005Metric, symbol Device:C
- removed FB5, FB7: 600R@100MHz, Inductor_SMD:L_0805_2012Metric, symbol Device:FerriteBead
- C54, C55: value 100nF -> 1uF; footprint Capacitor_SMD:C_0402_1005Metric -> Capacitor_SMD:C_0603_1608Metric
Connections:
- net OP_AMP+: now also C50.1, C52.1, D2.1 (K), R16.1, U5.23 (VPOS)
- net OP_AMP-: now also C47.2, C53.1, D3.2 (A), R19.1, U5.15 (VNEG)
Other:
- moved on the sheet: C55, C60, C62, C63, C64, C65, C66, C67, C68, C70, C71, C72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

Commit message: finished main
Parts:
- removed D1: LED, LED_SMD:LED_0603_1608Metric, symbol Device:LED
- removed R22: 100K, Resistor_SMD:R_0402_1005Metric, symbol Device:R
- removed R25: 47.5K, Resistor_SMD:R_0402_1005Metric, symbol Device:R
- added TP1, TP2, TP3, TP4, TP5: TestPoint, TestPoint:TestPoint_Pad_D2.5mm, symbol Connector:TestPoint
- FB4: value 600R@100MHz -> 120R@100MHz; footprint Inductor_SMD:L_0805_2012Metric -> Inductor_SMD:L_0603_1608Metric
- FB6: value 100R@100MHz -> 120R@100MHz; footprint Inductor_SMD:L_0805_2012Metric -> Inductor_SMD:L_0603_1608Metric
- R11: footprint Resistor_SMD:R_0402_1005Metric -> Resistor_SMD:R_0603_1608Metric
- R14: value 1K -> 10K
Connections:
- net +5V: now also TP2.1
- net OP_AMP+: now also TP3.1
- net OP_AMP-: now also TP4.1
- net V_SELECT: now also TP5.1; no longer R14.1
- net POWER_IND: now reaches U6.9 (ST)
- net POWER_IND: now also R14.2, TP1.1
- new net +3.3V: R14.1
- no-connect marks 0 -> 1

Commit message: manufactured
Parts:
- removed TP1: TestPoint, TestPoint:TestPoint_Pad_D2.5mm, symbol Connector:TestPoint
- TP2, TP3, TP4, TP5: footprint TestPoint:TestPoint_Pad_D2.5mm -> TestPoint:TestPoint_Pad_D2.0mm
Changed lines of the file:
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@@
 	)
 	(junction
-		(at 61.595 35.56)
-		(diameter 0)
-		(color 0 0 0 0)
-	)
-	(junction
 		(at 252.095 46.99)
 		(diameter 0)
@@
 	(wire
 		(pts
-			(xy 61.595 35.56) (xy 63.5 35.56)
+			(xy 60.96 35.56) (xy 63.5 35.56)
 		)
 		(stroke
@@
 	(wire
 		(pts
-			(xy 60.96 35.56) (xy 61.595 35.56)
-		)
-		(stroke
-			(width 0)
-			(type default)
-		)
-	)
-	(wire
-		(pts
 			(xy 78.105 95.885) (xy 86.995 95.885)
 		)
@@
 			)
 		)
-		(property "Footprint" "TestPoint:TestPoint_Pad_D2.5mm"
+		(property "Footprint" "TestPoint:TestPoint_Pad_D2.0mm"
 			(at 106.045 76.835 0)
 			(effects
@@
 			)
 		)
-		(property "Footprint" "TestPoint:TestPoint_Pad_D2.5mm"
+		(property "Footprint" "TestPoint:TestPoint_Pad_D2.0mm"
 			(at 92.71 26.67 0)
 			(effects
@@
 			)
 		)
-		(property "Footprint" "TestPoint:TestPoint_Pad_D2.5mm"
+		(property "Footprint" "TestPoint:TestPoint_Pad_D2.0mm"
 			(at 112.395 123.825 0)
 			(effects
@@
 	)
 	(symbol
-		(lib_id "Connector:TestPoint")
-		(at 61.595 35.56 0)
-		(unit 1)
-		(exclude_from_sim no)
-		(in_bom yes)
-		(on_board yes)
-		(dnp no)
-		(fields_autoplaced yes)
-		(property "Reference" "TP1"
-			(at 63.5 30.9879 0)
-			(effects
-				(font
-					(size 1.27 1.27)
-				)
-				(justify left)
-			)
-		)
-		(property "Value" "TestPoint"
-			(at 63.5 33.5279 0)
-			(effects
-				(font
-					(size 1.27 1.27)
-				)
-				(justify left)
-			)
-		)
-		(property "Footprint" "TestPoint:TestPoint_Pad_D2.5mm"
-			(at 66.675 35.56 0)
-			(effects
-				(font
-					(size 1.27 1.27)
-				)
-				(hide yes)
-			)
-		)
-		(property "Datasheet" "~"
-			(at 66.675 35.56 0)
-			(effects
-				(font
-					(size 1.27 1.27)
-				)
-				(hide yes)
-			)
-		)
-		(property "Description" "test point"
-			(at 61.595 35.56 0)
-			(effects
-				(font
-					(size 1.27 1.27)
-				)
-				(hide yes)
-			)
-		)
-		(pin "1"
-		)
-		(instances
-			(project ""
-				(path "/1061c21d-11bf-48d7-8db8-deedefa943c2/7d6e0902-de5f-4868-b5e7-4184774ee025"
-					(reference "TP1")
-					(unit 1)
-				)
-			)
-		)
-	)
-	(symbol
 		(lib_id "Device:R")
 		(at 210.185 60.96 0)
@@
 			)
 		)
-		(property "Footprint" "TestPoint:TestPoint_Pad_D2.5mm"
+		(property "Footprint" "TestPoint:TestPoint_Pad_D2.0mm"
 			(at 259.715 46.99 0)
 			(effects

Commit message: software unit testing
Connections:
- net +5V: no longer C66.2
- net at L3.1, U8.10 (SW): now also C66.2
Other:
- moved on the sheet: C66, R24, R26
Changed lines of the file:
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@@
 	)
 	(junction
+		(at 200.66 46.99)
+		(diameter 0)
+		(color 0 0 0 0)
+	)
+	(junction
 		(at 38.1 40.64)
 		(diameter 0)
@@
 	(wire
 		(pts
-			(xy 208.915 57.15) (xy 210.185 57.15)
-		)
-		(stroke
-			(width 0)
-			(type default)
-		)
-	)
-	(wire
-		(pts
 			(xy 94.615 160.02) (xy 94.615 162.56)
 		)
@@
 	(wire
 		(pts
-			(xy 226.695 36.83) (xy 199.39 36.83)
+			(xy 200.66 36.83) (xy 199.39 36.83)
 		)
 		(stroke
@@
 	(wire
 		(pts
-			(xy 226.695 39.37) (xy 226.695 36.83)
+			(xy 200.66 38.1) (xy 200.66 36.83)
 		)
 		(stroke
@@
 	(wire
 		(pts
+			(xy 200.66 46.99) (xy 207.645 46.99)
+		)
+		(stroke
+			(width 0)
+			(type default)
+		)
+	)
+	(wire
+		(pts
 			(xy 84.455 123.825) (xy 93.98 123.825)
 		)
@@
 	(wire
 		(pts
-			(xy 193.04 46.99) (xy 207.645 46.99)
+			(xy 193.04 46.99) (xy 200.66 46.99)
 		)
 		(stroke
@@
 	(wire
 		(pts
-			(xy 252.095 58.42) (xy 252.095 67.945)
+			(xy 252.095 61.595) (xy 252.095 67.945)
 		)
 		(stroke
@@
 	(wire
 		(pts
-			(xy 165.1 64.77) (xy 210.185 64.77)
+			(xy 165.1 64.77) (xy 208.915 64.77)
 		)
 		(stroke
@@
 	(wire
 		(pts
-			(xy 252.095 50.8) (xy 252.095 46.99)
+			(xy 252.095 53.975) (xy 252.095 46.99)
 		)
 		(stroke
@@
 	(wire
 		(pts
+			(xy 200.66 45.72) (xy 200.66 46.99)
+		)
+		(stroke
+			(width 0)
+			(type default)
+		)
+	)
+	(wire
+		(pts
 			(xy 93.98 111.125) (xy 93.98 116.205)
 		)
@@
 					(size 1.27 1.27)
 				)
+				(hide yes)
 			)
 		)
@@
 	(symbol
 		(lib_id "Device:R")
-		(at 210.185 60.96 0)
+		(at 208.915 60.96 0)
 		(unit 1)
 		(exclude_from_sim no)
@@
 		(fields_autoplaced yes)
 		(property "Reference" "R24"
-			(at 212.725 59.6899 0)
+			(at 211.455 59.6899 0)
 			(effects
 				(font
@@
 		)
 		(property "Value" "100K"
-			(at 212.725 62.2299 0)
+			(at 211.455 62.2299 0)
 			(effects
 				(font
@@
 		)
 		(property "Footprint" "Resistor_SMD:R_0402_1005Metric"
-			(at 208.407 60.96 90)
+			(at 207.137 60.96 90)
 			(effects
 				(font
@@
 		)
 		(property "Datasheet" "~"
-			(at 210.185 60.96 0)
+			(at 208.915 60.96 0)
 			(effects
 				(font
@@
 		)
 		(property "Description" "Resistor"
-			(at 210.185 60.96 0)
+			(at 208.915 60.96 0)
 			(effects
 				(font
@@
 	(symbol
 		(lib_id "Device:R")
-		(at 252.095 54.61 0)
+		(at 252.095 57.785 0)
 		(unit 1)
 		(exclude_from_sim no)
@@
 		(fields_autoplaced yes)
 		(property "Reference" "R26"
-			(at 254.635 53.3399 0)
+			(at 254.635 56.5149 0)
 			(effects
 				(font
@@
 		)
 		(property "Value" "30K"
-			(at 254.635 55.8799 0)
+			(at 254.635 59.0549 0)
 			(effects
 				(font
@@
 		)
 		(property "Footprint" "Resistor_SMD:R_0603_1608Metric"
-			(at 250.317 54.61 90)
+			(at 250.317 57.785 90)
 			(effects
 				(font
@@
 		)
 		(property "Datasheet" "~"
-			(at 252.095 54.61 0)
+			(at 252.095 57.785 0)
 			(effects
 				(font
@@
 		)
 		(property "Description" "Resistor"
-			(at 252.095 54.61 0)
+			(at 252.095 57.785 0)
 			(effects
 				(font
@@
 	(symbol
 		(lib_id "Device:C")
-		(at 226.695 43.18 0)
+		(at 200.66 41.91 0)
 		(unit 1)
 		(exclude_from_sim no)
@@
 		(dnp no)
 		(property "Reference" "C66"
-			(at 229.235 41.91 0)
+			(at 203.2 40.64 0)
 			(effects
 				(font
@@
 		)
 		(property "Value" "100nF"
-			(at 229.235 44.45 0)
+			(at 203.2 43.18 0)
 			(effects
 				(font
@@
 		)
 		(property "Footprint" "Capacitor_SMD:C_0402_1005Metric"
-			(at 227.6602 46.99 0)
+			(at 201.6252 45.72 0)
 			(effects
 				(font
@@
 		)
 		(property "Datasheet" "~"
-			(at 226.695 43.18 0)
+			(at 200.66 41.91 0)
 			(effects
 				(font
@@
 		)
 		(property "Description" "Unpolarized capacitor"
-			(at 226.695 43.18 0)
+			(at 200.66 41.91 0)
 			(effects
 				(font
