File: Electrical/Oscilliscope/OscilloscopeBoard/OscilloscopeBoard.kicad_sch (KiCad schematic)
At the start: 0 parts

Commit message: more usb debug
Parts:
- added U1: STM32G474RETx, Package_QFP:LQFP-64_10x10mm_P0.5mm, symbol MCU_ST_STM32G4:STM32G474RETx
Connections:
- new net: U1.1 (VBAT), U1.16 (VDD), U1.32 (VDD), U1.48 (VDD), U1.64 (VDD)
- new net: U1.15 (VSS), U1.31 (VSS), U1.47 (VSS), U1.63 (VSS)
