File: Electrical/FunctionGenerator/FuncGenBoard/FuncGenBoard.kicad_sch (KiCad schematic)
At the start: 0 parts

Commit message: function generator rough copy
Parts:
- added C1: 1uF, symbol Device:C
- added C10, C13, C14, C15, C4: 10uF, symbol Device:C
- added C11, C12, C2, C3, C5, C9: 100nF, symbol Device:C
- added C6: 10nF, symbol Device:C
- added C7, C8: 18pF, symbol Device:C
- added FB1, FB2, FB3: 600R@100MHz, symbol Device:FerriteBead
- added J1, J2: Conn_01x05_Socket, symbol Connector:Conn_01x05_Socket
- added R1: 1M, symbol Device:R
- added R2: 33, symbol Device:R
- added R3: 100k, symbol Device:R
- added R4: 1k, symbol Device:R
- added R5: 33k, symbol Device:R
- added R6: 50, symbol Device:R
- added U2: AD9833xRM, Package_SO:MSOP-10_3x3mm_P0.5mm, symbol Interface:AD9833xRM
- added U3: OPA2994xD, Package_SO:SOIC-8_3.9x4.9mm_P1.27mm, symbol Amplifier_Operational:OPA2994xD
- added U4: MCP41010, symbol Potentiometer_Digital:MCP41010
- added U5: 74LVC1GU04DRL, Package_TO_SOT_SMD:SOT-553, symbol 74xGxx:74LVC1GU04DRL
- added X1: X322525MOB4SI, Rocketry_Easyeda:CRYSTAL-SMD_4P-L3.2-W2.5-BL, symbol Rocketry_Easyeda:X322525MOB4SI
Connections:
- new net: C7.1, R1.1, U5.2, X1.1 (OSC1)
- new net: C8.1, R1.2, R2.2, U5.4, X1.3 (OSC2)
- new net: R5.2, R6.1, U3.7
- new net: U2.10 (VOUT), U4.5 (PA0)
- new net: U3.3 (+), U4.6 (PW0)
- new net: R4.1, R5.1, U3.6 (-)
- new net: C1.2, R3.1, U3.5 (+)
- new net: C2.1, C6.1, FB1.2, U2.2 (VDD)
- new net: C6.2, U2.1 (COMP)
- new net: C11.1, FB3.1, U3.8 (V+)
- new net: C5.1, U2.3 (CAP/2.5V)
- new net: R2.1, U2.5 (MCLK)
- new net: C12.1, FB2.2, U3.4 (V-)
- new net: C1.1, U3.1, U3.2 (-)
- new net +12V: C10.1, FB3.2, J1.5 (Pin_5)
- new net +3.3V: C14.1, C15.1, C3.1, C9.1, J1.3 (Pin_3), U4.8 (VDD), U5.5 (VCC)
- new net +3.3VA: C4.1, FB1.1, J1.2 (Pin_2)
- new net -12V: C13.1, FB2.1, J1.4 (Pin_4)
- new net CS_AD9833: J2.3 (Pin_3)
- new net CS_DIGIPOT: J2.2 (Pin_2), U4.1 (~{CS})
- new net GND: C10.2, C11.2, C12.2, C13.2, C14.2, C15.2, C2.2, C3.2, C4.2, C5.2, C7.2, C8.2, C9.2, J1.1 (Pin_1), J2.1 (Pin_1), R3.2, R4.2, U2.4 (DGND), U2.9 (AGND), U4.4 (VSS), U4.7 (PB0), U5.3 (GND), X1.2 (GND), X1.4 (GND)
- new net SCLK: J2.5 (Pin_5), U2.7 (SCLK), U4.2 (SCK)
- new net SDATA: J2.4 (Pin_4), U2.6 (SDATA), U4.3 (SI)
- new net V_Func: R6.2

Commit message: yolo
Parts:
- removed J1, J2: Conn_01x05_Socket, symbol Connector:Conn_01x05_Socket
- removed U3: OPA2994xD, Package_SO:SOIC-8_3.9x4.9mm_P1.27mm, symbol Amplifier_Operational:OPA2994xD
- removed U4: MCP41010, symbol Potentiometer_Digital:MCP41010
- removed U5: 74LVC1GU04DRL, Package_TO_SOT_SMD:SOT-553, symbol 74xGxx:74LVC1GU04DRL
- added C16, C18, C20: 100nF, Capacitor_SMD:C_0603_1608Metric, symbol Device:C
- added C17, C19, C21: 10uF, Capacitor_SMD:C_0805_2012Metric, symbol Device:C
- added C22: 100p, Capacitor_SMD:C_0603_1608Metric, symbol Device:C
- added D1: BAT54S, Package_TO_SOT_SMD:SOT-23, symbol Diode:BAT54S
- added FB4: 600R@100MHz, Inductor_SMD:L_0805_2012Metric, symbol Device:FerriteBead
- added H1, H2, H3, H4: MountingHole_Pad, MountingHole:MountingHole_3.2mm_M3_Pad_Via, symbol Mechanical:MountingHole_Pad
- added J1: Conn_01x02_Pin, Connector_PinHeader_2.54mm:PinHeader_1x02_P2.54mm_Vertical, symbol Connector:Conn_01x02_Pin
- added R10: 100k, Resistor_SMD:R_0603_1608Metric, symbol Device:R
- added R11: 50, Resistor_SMD:R_0603_1608Metric, symbol Device:R
- added R7: 330, Resistor_SMD:R_0603_1608Metric, symbol Device:R
- added R9: 1k, Resistor_SMD:R_0603_1608Metric, symbol Device:R
- added U14: SM08B-PASS-TBT(LF)(SN), JLC_Parts:CONN-SMD_SM08B-PASS-TBT-LF-SN, symbol JLC_PARTS:SM08B-PASS-TBT(LF)(SN)
- added U4, U7: MCP4151-xxxx-P, Package_SO:SOIC-8_3.9x4.9mm_P1.27mm, symbol Potentiometer_Digital:MCP4151-xxxx-P
- added U5: SN74LVC1GU04DBVR, Package_TO_SOT_SMD:SOT-23-5, symbol JLC_Parts:SN74LVC1GU04DBVR
- added U6: SM05B-PASS-TBT(LF)(SN), JLC_Parts:CONN-SMD_5P-P2.00_SM05B-PASS-TBT-LF-SN, symbol JLC_Parts:SM05B-PASS-TBT(LF)(SN)
- added U8: LM6172IMX/NOPB, Package_SO:SOIC-8_3.9x4.9mm_P1.27mm, symbol JLC_Parts:LM6172IMX/NOPB
- C1: value 1uF -> 100nF; footprint (none) -> Capacitor_SMD:C_0603_1608Metric
- C10, C13, C15, C4: footprint (none) -> Capacitor_SMD:C_0805_2012Metric
- C11, C12, C2, C3, C5, C6, C7, C8: footprint (none) -> Capacitor_SMD:C_0603_1608Metric
- C14: value 10uF -> 1uF; footprint (none) -> Capacitor_SMD:C_0603_1608Metric
- C9: value 100nF -> 10uF; footprint (none) -> Capacitor_SMD:C_0805_2012Metric
- FB1, FB2, FB3: footprint (none) -> Inductor_SMD:L_0805_2012Metric
- R1, R2: footprint (none) -> Resistor_SMD:R_0603_1608Metric
- R3: value 100k -> 100; footprint (none) -> Resistor_SMD:R_0603_1608Metric
- R4: value 1k -> 200; footprint (none) -> Resistor_SMD:R_0603_1608Metric
- R5: value 33k -> 1k; footprint (none) -> Resistor_SMD:R_0603_1608Metric
- R6: value 50 -> 5.6k; footprint (none) -> Resistor_SMD:R_0603_1608Metric
Connections:
- net +3.3VA is gone; now on net +3.3V: C4.1, FB1.1
- net +12V: now also D1.2 (K), U6.4
- net +3.3V: now also C1.1, C16.1, C17.1, C21.1, FB4.1, U14.7, U4.8 (V_{DD}), U5.5 (VCC), U6.1, U7.8 (V_{DD}); no longer C14.1
- net -12V: now also D1.1 (A), U6.5
- net CS_AD9833: now also U2.8 (~{FSYNC}), U14.4
- net GND: now also C1.2, R4.1, C16.2, C17.2, C18.2, C19.2, C20.2, C21.2, C22.2, H1.1, H2.1, H3.1, H4.1, J1.1 (Pin_1), R10.2, U14.10, U14.3, U14.8, U14.9, U4.4 (V_{SS}), U4.7 (P0B), U5.3 (GND), U6.2, U6.3, U6.6, U6.7, U7.4 (V_{SS}), U7.7 (P0B), U8.5 (INB+); no longer C14.2, R4.2
- net SCLK: now also U14.2, U4.2 (SCK), U7.2 (SCK)
- net SDATA: now also U14.1, U4.3 (SDI/SDO), U7.3 (SDI/SDO)
- net at C7.1, R1.1, X1.1 (OSC1): now also U5.2 (A)
- net at C8.1, R1.2, X1.3 (OSC2): now also R2.1, U5.4 (Y); no longer R2.2
- net A_OUT: now reaches R5.2
- net A_OUT: now also R3.1, R7.1, U8.2 (INA-); no longer R6.1
- net GEN_OUT: now reaches U2.10 (VOUT)
- net GEN_OUT: now also R4.2, C22.1, U4.5 (P0A)
- net at R5.1: now also U8.1 (OUTA); no longer R4.1
- net V+: now reaches C11.1, FB3.1
- net V+: now also U8.8 (V+)
- net MCLK: now reaches U2.5 (MCLK)
- net MCLK: now also R2.2; no longer R2.1
- net V-: now reaches C12.1, FB2.2
- net V-: now also R6.1, C18.1, C19.1, R7.2, R9.1, U8.4 (V-), U8.6 (INB-)
- net V_Func renamed DIGI_OFST
- net DIGI_OFST: now also U7.6 (P0W)
- new net: D1.3 (COM), J1.2 (Pin_2), R11.2
- new net: C14.2, U4.6 (P0W)
- new net 3.3_DIGI: C20.1, FB4.2, U7.5 (P0A)
- new net A_NINV: C14.1, R10.1, U8.3 (INA+)
- new net B_OUT: R11.1, R9.2, U8.7 (OUTB)
- new net CS_GAIN: U14.5, U4.1 (~{CS})
- new net CS_OFFSET: U14.6, U7.1 (~{CS})
- no-connect marks 0 -> 1
Other:
- note added: "25MHz CLOCK"
- note added: "DIGIPOT INPUT"
- note added: "DIGIPOTS"
- note added: "INPUT POWER"
- note added: "MOUNTING BOARD"
- note added: "OP-AMP RAILS"
- note added: "OUTPUT"
- note added: "STM GPIO PINS"
- note added: "WAVEGEN GAIN STAGE"
- note added: "WAVEGEN INITIAL STAGE"
- moved on the sheet: C10, C11, C12, C13, C15, C2, C3, C4, C7, C8, FB1, FB2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
